File: 1_hw/03_pcb/arb.kicad_sch (KiCad schematic)
At the start: 0 parts

Commit message: FEAT: Added USB ESD Protection.
Other:
- removed sheet POWER SEQUENCING
Changed lines of the file:
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@@
 	(text_box "TBD"
 		(exclude_from_sim no)
-		(at 165.1 88.9 0)
+		(at 165.1 85.09 0)
 		(size 19.05 3.81)
 		(stroke
@@
 	(text_box "TBD"
 		(exclude_from_sim no)
-		(at 165.1 92.71 0)
+		(at 165.1 88.9 0)
 		(size 19.05 3.81)
 		(stroke
@@
 	(text_box "TBD"
 		(exclude_from_sim no)
+		(at 165.1 100.33 0)
+		(size 19.05 3.81)
+		(stroke
+			(width 0)
+			(type default)
+			(color 0 0 0 1)
+		)
+		(fill
+			(type none)
+		)
+		(effects
+			(font
+				(size 1.27 1.27)
+				(color 0 72 72 1)
+			)
+		)
+	)
+	(text_box "TBD"
+		(exclude_from_sim no)
 		(at 165.1 104.14 0)
-		(size 19.05 3.81)
-		(stroke
-			(width 0)
-			(type default)
-			(color 0 0 0 1)
-		)
-		(fill
-			(type none)
-		)
-		(effects
-			(font
-				(size 1.27 1.27)
-				(color 0 72 72 1)
-			)
-		)
-	)
-	(text_box "TBD"
-		(exclude_from_sim no)
-		(at 165.1 107.95 0)
 		(size 19.05 3.81)
 		(stroke
@@
 	(text_box "TBD"
 		(exclude_from_sim no)
-		(at 165.1 100.33 0)
-		(size 19.05 3.81)
-		(stroke
-			(width 0)
-			(type default)
-			(color 0 0 0 1)
-		)
-		(fill
-			(type none)
-		)
-		(effects
-			(font
-				(size 1.27 1.27)
-				(color 0 72 72 1)
-			)
-		)
-	)
-	(text_box "TBD"
-		(exclude_from_sim no)
-		(at 165.1 85.09 0)
+		(at 165.1 96.52 0)
 		(size 19.05 3.81)
 		(stroke
@@
 	(text_box "TBD"
 		(exclude_from_sim no)
-		(at 165.1 115.57 0)
+		(at 165.1 111.76 0)
 		(size 19.05 3.81)
 		(stroke
@@
 	(text_box "TBD"
 		(exclude_from_sim no)
-		(at 165.1 96.52 0)
+		(at 165.1 92.71 0)
 		(size 19.05 3.81)
 		(stroke
@@
 	(text_box "TBD"
 		(exclude_from_sim no)
-		(at 165.1 111.76 0)
+		(at 165.1 107.95 0)
 		(size 19.05 3.81)
 		(stroke
@@
 	)
 	(sheet
+		(at 109.22 88.9)
+		(size 55.88 3.81)
+		(stroke
+			(width 0.1524)
+			(type solid)
+			(color 0 0 0 1)
+		)
+		(fill
+			(color 0 0 0 0.0000)
+		)
+		(property "Sheetname" "MICROPROCESSOR"
+			(at 110.236 90.932 0)
+			(effects
+				(font
+					(size 1.27 1.27)
+				)
+				(justify left)
+			)
+		)
+		(property "Sheetfile" "microprocessor.kicad_sch"
+			(at 109.22 93.2946 0)
+			(effects
+				(font
+					(size 1.27 1.27)
+				)
+				(justify left top)
+				(hide yes)
+			)
+		)
+		(instances
+			(project "arb"
+				(path "/866ef9be-3b01-4288-a6e0-a2357aa17e50"
+					(page "5")
+				)
+			)
+		)
+	)
+	(sheet
 		(at 109.22 92.71)
 		(size 55.88 3.81)
@@
 			(color 0 0 0 0.0000)
 		)
-		(property "Sheetname" "MICROPROCESSOR"
+		(property "Sheetname" "FPGA"
 			(at 110.236 94.742 0)
 			(effects
@@
 			)
 		)
-		(property "Sheetfile" "microprocessor.kicad_sch"
+		(property "Sheetfile" "fpga.kicad_sch"
 			(at 109.22 97.1046 0)
 			(effects
@@
 			(project "arb"
 				(path "/866ef9be-3b01-4288-a6e0-a2357aa17e50"
-					(page "5")
-				)
-			)
-		)
-	)
-	(sheet
-		(at 109.22 96.52)
-		(size 55.88 3.81)
-		(stroke
-			(width 0.1524)
-			(type solid)
-			(color 0 0 0 1)
-		)
-		(fill
-			(color 0 0 0 0.0000)
-		)
-		(property "Sheetname" "FPGA"
-			(at 110.236 98.552 0)
-			(effects
-				(font
-					(size 1.27 1.27)
-				)
-				(justify left)
-			)
-		)
-		(property "Sheetfile" "fpga.kicad_sch"
-			(at 109.22 100.9146 0)
-			(effects
-				(font
-					(size 1.27 1.27)
-				)
-				(justify left top)
-				(hide yes)
-			)
-		)
-		(instances
-			(project "arb"
-				(path "/866ef9be-3b01-4288-a6e0-a2357aa17e50"
 					(page "6")
 				)
@@
 	)
 	(sheet
-		(at 109.22 107.95)
+		(at 109.22 104.14)
 		(size 55.88 3.81)
 		(stroke
@@
 		)
 		(property "Sheetname" "ANALOG - STAGE 1"
-			(at 110.236 109.982 0)
+			(at 110.236 106.172 0)
 			(effects
 				(font
@@
 		)
 		(property "Sheetfile" "analog1.kicad_sch"
-			(at 109.22 112.3446 0)
+			(at 109.22 108.5346 0)
 			(effects
 				(font
@@
 			(color 0 0 0 0.0000)
 		)
-		(property "Sheetname" "POWER SEQUENCING"
+		(property "Sheetname" "CLOCKING"
 			(at 110.236 87.122 0)
 			(effects
@@
 			)
 		)
-		(property "Sheetfile" "power_seq.kicad_sch"
+		(property "Sheetfile" "clocking.kicad_sch"
 			(at 109.22 89.4846 0)
 			(effects
@@
 			(project "arb"
 				(path "/866ef9be-3b01-4288-a6e0-a2357aa17e50"
-					(page "3")
-				)
-			)
-		)
-	)
-	(sheet
-		(at 109.22 88.9)
-		(size 55.88 3.81)
-		(stroke
-			(width 0.1524)
-			(type solid)
-			(color 0 0 0 1)
-		)
-		(fill
-			(color 0 0 0 0.0000)
-		)
-		(property "Sheetname" "CLOCKING"
-			(at 110.236 90.932 0)
-			(effects
-				(font
-					(size 1.27 1.27)
-				)
-				(justify left)
-			)
-		)
-		(property "Sheetfile" "clocking.kicad_sch"
-			(at 109.22 93.2946 0)
-			(effects
-				(font
-					(size 1.27 1.27)
-				)
-				(justify left top)
-				(hide yes)
-			)
-		)
-		(instances
-			(project "arb"
-				(path "/866ef9be-3b01-4288-a6e0-a2357aa17e50"
 					(page "4")
 				)
@@
 	)
 	(sheet
+		(at 109.22 96.52)
+		(size 55.88 3.81)
+		(stroke
+			(width 0.1524)
+			(type solid)
+			(color 0 0 0 1)
+		)
+		(fill
+			(color 0 0 0 0.0000)
+		)
+		(property "Sheetname" "FTDI"
+			(at 110.236 98.552 0)
+			(effects
+				(font
+					(size 1.27 1.27)
+				)
+				(justify left)
+			)
+		)
+		(property "Sheetfile" "ftdi.kicad_sch"
+			(at 109.22 100.9146 0)
+			(effects
+				(font
+					(size 1.27 1.27)
+				)
+				(justify left top)
+				(hide yes)
+			)
+		)
+		(instances
+			(project "arb"
+				(path "/866ef9be-3b01-4288-a6e0-a2357aa17e50"
+					(page "7")
+				)
+			)
+		)
+	)
+	(sheet
 		(at 109.22 100.33)
 		(size 55.88 3.81)
@@
 			(color 0 0 0 0.0000)
 		)
-		(property "Sheetname" "FTDI"
+		(property "Sheetname" "DAC"
 			(at 110.236 102.362 0)
 			(effects
@@
 			)
 		)
-		(property "Sheetfile" "ftdi.kicad_sch"
+		(property "Sheetfile" "dac.kicad_sch"
 			(at 109.22 104.7246 0)
-			(effects
-				(font
-					(size 1.27 1.27)
-				)
-				(justify left top)
-				(hide yes)
-			)
-		)
-		(instances
-			(project "arb"
-				(path "/866ef9be-3b01-4288-a6e0-a2357aa17e50"
-					(page "7")
-				)
-			)
-		)
-	)
-	(sheet
-		(at 109.22 104.14)
-		(size 55.88 3.81)
-		(stroke
-			(width 0.1524)
-			(type solid)
-			(color 0 0 0 1)
-		)
-		(fill
-			(color 0 0 0 0.0000)
-		)
-		(property "Sheetname" "DAC"
-			(at 110.236 106.172 0)
-			(effects
-				(font
-					(size 1.27 1.27)
-				)
-				(justify left)
-			)
-		)
-		(property "Sheetfile" "dac.kicad_sch"
-			(at 109.22 108.5346 0)
 			(effects
 				(font
@@
 	)
 	(sheet
-		(at 109.22 115.57)
+		(at 109.22 111.76)
 		(size 55.88 3.81)
 		(stroke
@@
 		)
 		(property "Sheetname" "ANALOG - DC OFFSET"
-			(at 110.236 117.602 0)
+			(at 110.236 113.792 0)
 			(effects
 				(font
@@
 		)
 		(property "Sheetfile" "analogdc.kicad_sch"
-			(at 109.22 119.9646 0)
+			(at 109.22 116.1546 0)
 			(effects
 				(font
@@
 	)
 	(sheet
-		(at 109.22 111.76)
+		(at 109.22 107.95)
 		(size 55.88 3.81)
 		(stroke
@@
 		)
 		(property "Sheetname" "ANALOG - STAGE 2"
-			(at 110.236 113.792 0)
+			(at 110.236 109.982 0)
 			(effects
 				(font
@@
 		)
 		(property "Sheetfile" "analog2.kicad_sch"
-			(at 109.22 116.1546 0)
-			(effects
-				(font
+			(at 109.22 112.3446 0)
+			(effects
+				(font

Commit message: FEAT: Assigned Reference Designators; Assigned Passives Part Numbers & Footprints (0603); Assigned LCSC P/Ns.
Changed lines of the file:
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@@
 		)
 	)
-	(text_box "TBD"
+	(text_box "3"
 		(exclude_from_sim no)
 		(at 165.1 85.09 0)
@@
 		)
 	)
-	(text_box "TBD"
+	(text_box "4"
 		(exclude_from_sim no)
 		(at 165.1 88.9 0)
@@
 		)
 	)
-	(text_box "TBD"
+	(text_box "7"
 		(exclude_from_sim no)
 		(at 165.1 100.33 0)
@@
 		)
 	)
-	(text_box "TBD"
+	(text_box "8"
 		(exclude_from_sim no)
 		(at 165.1 104.14 0)
@@
 		)
 	)
-	(text_box "TBD"
-		(exclude_from_sim no)
-		(at 165.1 135.89 0)
+	(text_box "11"
+		(exclude_from_sim no)
+		(at 165.1 115.57 0)
 		(size 19.05 3.81)
 		(stroke
@@
 		)
 	)
-	(text_box "TBD"
+	(text_box "6"
 		(exclude_from_sim no)
 		(at 165.1 96.52 0)
@@
 		)
 	)
-	(text_box "TBD"
+	(text_box "10"
 		(exclude_from_sim no)
 		(at 165.1 111.76 0)
@@
 		)
 	)
-	(text_box "TBD"
+	(text_box "5"
 		(exclude_from_sim no)
 		(at 165.1 92.71 0)
@@
 		)
 	)
-	(text_box "TBD"
+	(text_box "9"
 		(exclude_from_sim no)
 		(at 165.1 107.95 0)
@@
 	(text "NOTE: USED TO COPY & PASTE A BLANK HIERARCHAL SCHEMATIC SHEET."
 		(exclude_from_sim no)
-		(at 144.018 149.606 0)
+		(at 144.018 213.106 0)
 		(effects
 			(font
@@
 			(project "arb"
 				(path "/866ef9be-3b01-4288-a6e0-a2357aa17e50"
-					(page "5")
+					(page "4")
 				)
 			)
@@
 			(project "arb"
 				(path "/866ef9be-3b01-4288-a6e0-a2357aa17e50"
-					(page "6")
+					(page "5")
 				)
 			)
@@
 			(project "arb"
 				(path "/866ef9be-3b01-4288-a6e0-a2357aa17e50"
-					(page "10")
+					(page "8")
 				)
 			)
@@
 			(project "arb"
 				(path "/866ef9be-3b01-4288-a6e0-a2357aa17e50"
-					(page "4")
+					(page "3")
 				)
 			)
@@
 			(project "arb"
 				(path "/866ef9be-3b01-4288-a6e0-a2357aa17e50"
-					(page "7")
+					(page "6")
 				)
 			)
@@
 			(project "arb"
 				(path "/866ef9be-3b01-4288-a6e0-a2357aa17e50"
-					(page "8")
-				)
-			)
-		)
-	)
-	(sheet
-		(at 109.22 151.13)
+					(page "7")
+				)
+			)
+		)
+	)
+	(sheet
+		(at 109.22 214.63)
 		(size 55.88 3.81)
 		(stroke
@@
 		)
 		(property "Sheetname" "BLANK TEMPLATE"
-			(at 110.236 153.162 0)
+			(at 110.236 216.662 0)
 			(effects
 				(font
@@
 		)
 		(property "Sheetfile" "blank_template.kicad_sch"
-			(at 109.22 155.5246 0)
+			(at 109.22 219.0246 0)
 			(effects
 				(font
@@
 			(project "arb"
 				(path "/866ef9be-3b01-4288-a6e0-a2357aa17e50"
-					(page "12")
+					(page "10")
 				)
 			)
@@
 			(project "arb"
 				(path "/866ef9be-3b01-4288-a6e0-a2357aa17e50"
+					(page "9")
+				)
+			)
+		)
+	)
+	(sheet
+		(at 109.22 115.57)
+		(size 55.88 3.81)
+		(stroke
+			(width 0.1524)
+			(type solid)
+			(color 0 0 0 1)
+		)
+		(fill
+			(color 0 0 0 0.0000)
+		)
+		(property "Sheetname" "CONNECTORS"
+			(at 110.236 117.602 0)
+			(effects
+				(font
+					(size 1.27 1.27)
+				)
+				(justify left)
+			)
+		)
+		(property "Sheetfile" "connectors.kicad_sch"
+			(at 109.22 119.9646 0)
+			(effects
+				(font
+					(size 1.27 1.27)
+				)
+				(justify left top)
+				(hide yes)
+			)
+		)
+		(instances
+			(project "arb"
+				(path "/866ef9be-3b01-4288-a6e0-a2357aa17e50"
 					(page "11")
 				)
 			)
-		)
-	)
-	(sheet
-		(at 109.22 135.89)
-		(size 55.88 3.81)
-		(stroke
-			(width 0.1524)
-			(type solid)
-			(color 0 0 0 1)
-		)
-		(fill
-			(color 0 0 0 0.0000)
-		)
-		(property "Sheetname" "CONNECTORS"
-			(at 110.236 137.922 0)
-			(effects
-				(font
-					(size 1.27 1.27)
-				)
-				(justify left)
-			)
-		)
-		(property "Sheetfile" "connectors.kicad_sch"
-			(at 109.22 140.2846 0)
-			(effects
-				(font
-					(size 1.27 1.27)
-				)
-				(justify left top)
-				(hide yes)
-			)
-		)
-		(instances
-			(project "arb"
-				(path "/866ef9be-3b01-4288-a6e0-a2357aa17e50"
-					(page "20")
-				)
-			)

Commit message: FEAT: Added MCU Flash. Finished creating & assigning footprints. Ran ERC & cleared out issues. Ready for Layout.
Other:
- added sheet FLASH (flash.kicad_sch)
Changed lines of the file:
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@@
+		)
+	)
+	(text_box "12"
+		(exclude_from_sim no)
+		(at 165.1 119.38 0)
+		(size 19.05 3.81)
+		(stroke
+			(width 0)
+			(type default)
+			(color 0 0 0 1)
+		)
+		(fill
+			(type none)
+		)
+		(effects
+			(font
+				(size 1.27 1.27)
+				(color 0 72 72 1)
+			)
 		)
 	)
@@
 	)
 	(sheet
-		(at 109.22 104.14)
+		(at 109.22 107.95)
 		(size 55.88 3.81)
 		(stroke
@@
 		)
 		(property "Sheetname" "ANALOG - STAGE 1"
-			(at 110.236 106.172 0)
+			(at 110.236 109.982 0)
 			(effects
 				(font
@@
 		)
 		(property "Sheetfile" "analog1.kicad_sch"
-			(at 109.22 108.5346 0)
-			(effects
-				(font
-					(size 1.27 1.27)
-				)
-				(justify left top)
-				(hide yes)
-			)
-		)
-		(instances
-			(project "arb"
-				(path "/866ef9be-3b01-4288-a6e0-a2357aa17e50"
-					(page "8")
+			(at 109.22 112.3446 0)
+			(effects
+				(font
+					(size 1.27 1.27)
+				)
+				(justify left top)
+				(hide yes)
+			)
+		)
+		(instances
+			(project "arb"
+				(path "/866ef9be-3b01-4288-a6e0-a2357aa17e50"
+					(page "9")
 				)
 			)
@@
 	)
 	(sheet
+		(at 109.22 96.52)
+		(size 55.88 3.81)
+		(stroke
+			(width 0.1524)
+			(type solid)
+			(color 0 0 0 1)
+		)
+		(fill
+			(color 0 0 0 0.0000)
+		)
+		(property "Sheetname" "FLASH"
+			(at 110.236 98.552 0)
+			(effects
+				(font
+					(size 1.27 1.27)
+				)
+				(justify left)
+			)
+		)
+		(property "Sheetfile" "flash.kicad_sch"
+			(at 109.22 100.9146 0)
+			(effects
+				(font
+					(size 1.27 1.27)
+				)
+				(justify left top)
+				(hide yes)
+			)
+		)
+		(instances
+			(project "arb"
+				(path "/866ef9be-3b01-4288-a6e0-a2357aa17e50"
+					(page "7")
+				)
+			)
+		)
+	)
+	(sheet
 		(at 109.22 85.09)
 		(size 55.88 3.81)
@@
 	)
 	(sheet
-		(at 109.22 96.52)
+		(at 109.22 100.33)
 		(size 55.88 3.81)
 		(stroke
@@
 		)
 		(property "Sheetname" "FTDI"
-			(at 110.236 98.552 0)
+			(at 110.236 102.362 0)
 			(effects
 				(font
@@
 		)
 		(property "Sheetfile" "ftdi.kicad_sch"
-			(at 109.22 100.9146 0)
+			(at 109.22 104.7246 0)
 			(effects
 				(font
@@
 	)
 	(sheet
-		(at 109.22 100.33)
+		(at 109.22 104.14)
 		(size 55.88 3.81)
 		(stroke
@@
 		)
 		(property "Sheetname" "DAC"
-			(at 110.236 102.362 0)
+			(at 110.236 106.172 0)
 			(effects
 				(font
@@
 		)
 		(property "Sheetfile" "dac.kicad_sch"
-			(at 109.22 104.7246 0)
-			(effects
-				(font
-					(size 1.27 1.27)
-				)
-				(justify left top)
-				(hide yes)
-			)
-		)
-		(instances
-			(project "arb"
-				(path "/866ef9be-3b01-4288-a6e0-a2357aa17e50"
-					(page "7")
+			(at 109.22 108.5346 0)
+			(effects
+				(font
+					(size 1.27 1.27)
+				)
+				(justify left top)
+				(hide yes)
+			)
+		)
+		(instances
+			(project "arb"
+				(path "/866ef9be-3b01-4288-a6e0-a2357aa17e50"
+					(page "8")
 				)
 			)
@@
 	)
 	(sheet
+		(at 109.22 115.57)
+		(size 55.88 3.81)
+		(stroke
+			(width 0.1524)
+			(type solid)
+			(color 0 0 0 1)
+		)
+		(fill
+			(color 0 0 0 0.0000)
+		)
+		(property "Sheetname" "ANALOG - DC OFFSET"
+			(at 110.236 117.602 0)
+			(effects
+				(font
+					(size 1.27 1.27)
+				)
+				(justify left)
+			)
+		)
+		(property "Sheetfile" "analogdc.kicad_sch"
+			(at 109.22 119.9646 0)
+			(effects
+				(font
+					(size 1.27 1.27)
+				)
+				(justify left top)
+				(hide yes)
+			)
+		)
+		(instances
+			(project "arb"
+				(path "/866ef9be-3b01-4288-a6e0-a2357aa17e50"
+					(page "11")
+				)
+			)
+		)
+	)
+	(sheet
 		(at 109.22 111.76)
 		(size 55.88 3.81)
@@
 			(color 0 0 0 0.0000)
 		)
-		(property "Sheetname" "ANALOG - DC OFFSET"
+		(property "Sheetname" "ANALOG - STAGE 2"
 			(at 110.236 113.792 0)
 			(effects
@@
 			)
 		)
-		(property "Sheetfile" "analogdc.kicad_sch"
+		(property "Sheetfile" "analog2.kicad_sch"
 			(at 109.22 116.1546 0)
 			(effects
@@
 	)
 	(sheet
-		(at 109.22 107.95)
-		(size 55.88 3.81)
-		(stroke
-			(width 0.1524)
-			(type solid)
-			(color 0 0 0 1)
-		)
-		(fill
-			(color 0 0 0 0.0000)
-		)
-		(property "Sheetname" "ANALOG - STAGE 2"
-			(at 110.236 109.982 0)
-			(effects
-				(font
-					(size 1.27 1.27)
-				)
-				(justify left)
-			)
-		)
-		(property "Sheetfile" "analog2.kicad_sch"
-			(at 109.22 112.3446 0)
-			(effects
-				(font
-					(size 1.27 1.27)
-				)
-				(justify left top)
-				(hide yes)
-			)
-		)
-		(instances
-			(project "arb"
-				(path "/866ef9be-3b01-4288-a6e0-a2357aa17e50"
-					(page "9")
-				)
-			)
-		)
-	)
-	(sheet
-		(at 109.22 115.57)
+		(at 109.22 119.38)
 		(size 55.88 3.81)
 		(stroke
@@
 		)
 		(property "Sheetname" "CONNECTORS"
-			(at 110.236 117.602 0)
+			(at 110.236 121.412 0)
 			(effects
 				(font
@@
 		)
 		(property "Sheetfile" "connectors.kicad_sch"
-			(at 109.22 119.9646 0)
-			(effects
-				(font
-					(size 1.27 1.27)
-				)
-				(justify left top)
-				(hide yes)
-			)
-		)
-		(instances
-			(project "arb"
-				(path "/866ef9be-3b01-4288-a6e0-a2357aa17e50"
-					(page "11")
-				)
-			)
+			(at 109.22 123.7746 0)
+			(effects
+				(font
+					(size 1.27 1.27)
+				)
+				(justify left top)
+				(hide yes)
+			)
+		)
+		(instances
+			(project "arb"
+				(path "/866ef9be-3b01-4288-a6e0-a2357aa17e50"
+					(page "12")
+				)
+			)
