File: 1_hw/03_pcb/clocking.kicad_sch (KiCad schematic)
At the start: 23 parts, among them U12 ADG1219BRJZ, U13 LMK1C1103PWR, X1 ASE-10.000MHz, X2 ASE-100.000MHz

Commit message: FEAT: Assigned Reference Designators; Assigned Passives Part Numbers & Footprints (0603); Assigned LCSC P/Ns.
Parts:
- C33: renamed from C69; LCSC (none) -> C24452; PN CL10B104JB8NNNC -> (none); Part Number (none) -> CL10B104JB8NNNC
- C34: renamed from C70; LCSC (none) -> C24452; PN CL10B104JB8NNNC -> (none); Part Number (none) -> CL10B104JB8NNNC
- C35: renamed from C71; LCSC (none) -> C24452; PN CL10B104JB8NNNC -> (none); Part Number (none) -> CL10B104JB8NNNC
- C36: renamed from C72; LCSC (none) -> C24452; PN CL10B104JB8NNNC -> (none); Part Number (none) -> CL10B104JB8NNNC
- C37: renamed from C73; footprint (none) -> Capacitor_SMD:C_0603_1608Metric; LCSC (none) -> C327203; Part Number (none) -> CC0603CRNPO9BN5R0
- FB1: LCSC (none) -> C491555
- FB2: LCSC (none) -> C491547
- R18: renamed from R28; LCSC (none) -> C25804; PN CR-03FC7---10K -> (none); Part Number (none) -> 0603WAF1002T5E
- R19: renamed from R29; value 25 -> 24.9; LCSC (none) -> C22916; Part Number (none) -> 0603WAF249JT5E
- R20: renamed from R30; LCSC (none) -> C25804; PN CR-03FC7---10K -> (none); Part Number (none) -> 0603WAF1002T5E
- R21: renamed from R31; value 25 -> 24.9; LCSC (none) -> C22916; Part Number (none) -> 0603WAF249JT5E
- R22: renamed from R32; LCSC (none) -> C25804; PN CR-03FC7---10K -> (none); Part Number (none) -> 0603WAF1002T5E
- R23: renamed from R33; LCSC (none) -> C25804; PN CR-03FC7---10K -> (none); Part Number (none) -> 0603WAF1002T5E
- R24: renamed from R34; LCSC (none) -> C25804; PN CR-03FC7---10K -> (none); Part Number (none) -> 0603WAF1002T5E
- R25: renamed from R35; footprint (none) -> Resistor_SMD:R_0603_1608Metric; LCSC (none) -> C105588; Part Number (none) -> RC0603FR-07100RL
- R26: renamed from R36; footprint (none) -> Resistor_SMD:R_0603_1608Metric; LCSC (none) -> C105588; Part Number (none) -> RC0603FR-07100RL
- R27: renamed from R37; value 25 -> 24.9; LCSC (none) -> C22916; Part Number (none) -> 0603WAF249JT5E
- R28: renamed from R38; value 25 -> 24.9; LCSC (none) -> C22916; Part Number (none) -> 0603WAF249JT5E
- R29: renamed from R39; LCSC (none) -> C15402; Part Number (none) -> 0603WAJ0000T5E
- U10: renamed from U13; LCSC (none) -> C2873274
- U9: renamed from U12; footprint BRZK_TBD -> (none); LCSC (none) -> C579007
- X1: Part Number (none) -> ASE-10.000MHz
- X2: Part Number (none) -> ASE-100.000MHz

Commit message: FEAT: Added MCU Flash. Finished creating & assigning footprints. Ran ERC & cleared out issues. Ready for Layout.
Parts:
- FB1, FB2: footprint (none) -> Inductor_SMD:L_0603_1608Metric
- U9: footprint (none) -> Package_TO_SOT_SMD:SOT-23-8
- renumbered R18 to R19, R19 to R20, R20 to R21, R21 to R22, R22 to R23, R23 to R24, R24 to R25, R25 to R26, R26 to R27, R27 to R28, R28 to R29, R29 to R30
