File: 1_hw/03_pcb/flash.kicad_sch (KiCad schematic)
At the start: 8 parts, among them U15 W25Q128JVSIQ, U16 W25Q128JVSIQ

Commit message: MINOR: Verified Footprints to Datasheets. Added Pull Ups on FPGA DONE/Config/SPI Chip Select Pins.
Parts:
- renumbered R50 to R53, R51 to R54, R52 to R55, R53 to R56
Changed lines of the file:
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@@
 		(dnp no)
 		(fields_autoplaced yes)
-		(property "Reference" "#PWR0206"
+		(property "Reference" "#PWR0209"
 			(at 156.21 105.41 0)
 			(effects
@@
 			(project "arb"
 				(path "/866ef9be-3b01-4288-a6e0-a2357aa17e50/3eaf535e-ef91-4de7-bf25-42486b2f88fe"
-					(reference "#PWR0206")
+					(reference "#PWR0209")
 					(unit 1)
 				)
@@
 		(on_board yes)
 		(dnp no)
-		(property "Reference" "R51"
+		(property "Reference" "R54"
 			(at 127.762 134.366 0)
 			(effects
@@
 			(project "arb"
 				(path "/866ef9be-3b01-4288-a6e0-a2357aa17e50/3eaf535e-ef91-4de7-bf25-42486b2f88fe"
-					(reference "R51")
+					(reference "R54")
 					(unit 1)
 				)
@@
 		(dnp no)
 		(fields_autoplaced yes)
-		(property "Reference" "#PWR0210"
+		(property "Reference" "#PWR0213"
 			(at 162.56 137.16 0)
 			(effects
@@
 			(project "arb"
 				(path "/866ef9be-3b01-4288-a6e0-a2357aa17e50/3eaf535e-ef91-4de7-bf25-42486b2f88fe"
-					(reference "#PWR0210")
+					(reference "#PWR0213")
 					(unit 1)
 				)
@@
 		(dnp no)
 		(fields_autoplaced yes)
-		(property "Reference" "#PWR0205"
+		(property "Reference" "#PWR0208"
 			(at 156.21 66.04 0)
 			(effects
@@
 			(project "arb"
 				(path "/866ef9be-3b01-4288-a6e0-a2357aa17e50/3eaf535e-ef91-4de7-bf25-42486b2f88fe"
-					(reference "#PWR0205")
+					(reference "#PWR0208")
 					(unit 1)
 				)
@@
 		(dnp no)
 		(fields_autoplaced yes)
-		(property "Reference" "#PWR0209"
+		(property "Reference" "#PWR0212"
 			(at 161.29 76.2 0)
 			(effects
@@
 			(project "arb"
 				(path "/866ef9be-3b01-4288-a6e0-a2357aa17e50/3eaf535e-ef91-4de7-bf25-42486b2f88fe"
-					(reference "#PWR0209")
+					(reference "#PWR0212")
 					(unit 1)
 				)
@@
 		(on_board yes)
 		(dnp no)
-		(property "Reference" "R53"
+		(property "Reference" "R56"
 			(at 136.652 134.366 0)
 			(effects
@@
 			(project "arb"
 				(path "/866ef9be-3b01-4288-a6e0-a2357aa17e50/3eaf535e-ef91-4de7-bf25-42486b2f88fe"
-					(reference "R53")
+					(reference "R56")
 					(unit 1)
 				)
@@
 		(dnp no)
 		(fields_autoplaced yes)
-		(property "Reference" "#PWR0207"
+		(property "Reference" "#PWR0210"
 			(at 157.48 127 0)
 			(effects
@@
 			(project "arb"
 				(path "/866ef9be-3b01-4288-a6e0-a2357aa17e50/3eaf535e-ef91-4de7-bf25-42486b2f88fe"
-					(reference "#PWR0207")
+					(reference "#PWR0210")
 					(unit 1)
 				)
@@
 		(on_board yes)
 		(dnp no)
-		(property "Reference" "R50"
+		(property "Reference" "R53"
 			(at 126.492 73.406 0)
 			(effects
@@
 			(project "arb"
 				(path "/866ef9be-3b01-4288-a6e0-a2357aa17e50/3eaf535e-ef91-4de7-bf25-42486b2f88fe"
-					(reference "R50")
+					(reference "R53")
 					(unit 1)
 				)
@@
 		(on_board yes)
 		(dnp no)
-		(property "Reference" "R52"
+		(property "Reference" "R55"
 			(at 135.382 73.406 0)
 			(effects
@@
 			(project "arb"
 				(path "/866ef9be-3b01-4288-a6e0-a2357aa17e50/3eaf535e-ef91-4de7-bf25-42486b2f88fe"
-					(reference "R52")
+					(reference "R55")
 					(unit 1)
 				)
@@
 		(dnp no)
 		(fields_autoplaced yes)
-		(property "Reference" "#PWR0204"
+		(property "Reference" "#PWR0207"
 			(at 142.24 137.16 0)
 			(effects
@@
 			(project "arb"
 				(path "/866ef9be-3b01-4288-a6e0-a2357aa17e50/3eaf535e-ef91-4de7-bf25-42486b2f88fe"
-					(reference "#PWR0204")
+					(reference "#PWR0207")
 					(unit 1)
 				)
@@
 		(dnp no)
 		(fields_autoplaced yes)
-		(property "Reference" "#PWR0202"
+		(property "Reference" "#PWR0205"
 			(at 133.35 137.16 0)
 			(effects
@@
 			(project "arb"
 				(path "/866ef9be-3b01-4288-a6e0-a2357aa17e50/3eaf535e-ef91-4de7-bf25-42486b2f88fe"
-					(reference "#PWR0202")
+					(reference "#PWR0205")
 					(unit 1)
 				)
@@
 		(dnp no)
 		(fields_autoplaced yes)
-		(property "Reference" "#PWR0208"
+		(property "Reference" "#PWR0211"
 			(at 157.48 166.37 0)
 			(effects
@@
 			(project "arb"
 				(path "/866ef9be-3b01-4288-a6e0-a2357aa17e50/3eaf535e-ef91-4de7-bf25-42486b2f88fe"
-					(reference "#PWR0208")
+					(reference "#PWR0211")
 					(unit 1)
 				)
@@
 		(dnp no)
 		(fields_autoplaced yes)
-		(property "Reference" "#PWR0201"
+		(property "Reference" "#PWR0204"
 			(at 132.08 76.2 0)
 			(effects
@@
 			(project "arb"
 				(path "/866ef9be-3b01-4288-a6e0-a2357aa17e50/3eaf535e-ef91-4de7-bf25-42486b2f88fe"
-					(reference "#PWR0201")
+					(reference "#PWR0204")
 					(unit 1)
 				)
@@
 		(dnp no)
 		(fields_autoplaced yes)
-		(property "Reference" "#PWR0203"
+		(property "Reference" "#PWR0206"
 			(at 140.97 76.2 0)
 			(effects
@@
 			(project "arb"
 				(path "/866ef9be-3b01-4288-a6e0-a2357aa17e50/3eaf535e-ef91-4de7-bf25-42486b2f88fe"
-					(reference "#PWR0203")
-					(unit 1)
-				)
+					(reference "#PWR0206")
+					(unit 1)
+				)
