File: 1_hw/03_pcb/analog1.kicad_sch (KiCad schematic)
At the start: 26 parts, among them U19 LM6171, U20 LM6171, U21 TMUX6104

Commit message: MINOR: Verified Footprints to Datasheets. Added Pull Ups on FPGA DONE/Config/SPI Chip Select Pins.
Parts:
- renumbered R57 to R60, R58 to R61, R59 to R62, R60 to R63, R61 to R64, R62 to R65, R63 to R66, R64 to R67, R65 to R68, R66 to R69, R67 to R70, R68 to R71, R69 to R72, R70 to R73, R71 to R74

Commit message: FEAT: Initial board placement started.
Parts:
- C94: renamed from C89; now not fitted
- renumbered C95 to C100, C96 to C101, C90 to C95, C91 to C96, C92 to C97, C93 to C98, C94 to C99
Connections:
- net 15P0V_A: now also U21.12 (VDD); no longer U21.13 (VDD)
- net GND: now also U21.13 (GND); no longer U21.14 (A1)
Changed lines of the file:
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@@
 		(on_board yes)
 		(dnp no)
-		(property "Reference" "#PWR0233"
+		(property "Reference" "#PWR0245"
 			(at 100.33 39.37 0)
 			(effects
@@
 			(project "arb"
 				(path "/866ef9be-3b01-4288-a6e0-a2357aa17e50/15631b2d-3708-4ae8-a4e9-7f8a7b587733"
-					(reference "#PWR0233")
+					(reference "#PWR0245")
 					(unit 1)
 				)
@@
 		(in_bom yes)
 		(on_board yes)
-		(dnp no)
+		(dnp yes)
 		(fields_autoplaced yes)
-		(property "Reference" "C89"
+		(property "Reference" "C94"
 			(at 63.5063 39.37 90)
 			(effects
@@
 			(project ""
 				(path "/866ef9be-3b01-4288-a6e0-a2357aa17e50/15631b2d-3708-4ae8-a4e9-7f8a7b587733"
-					(reference "C89")
+					(reference "C94")
 					(unit 1)
 				)
@@
 		(dnp no)
 		(fields_autoplaced yes)
-		(property "Reference" "#PWR0231"
+		(property "Reference" "#PWR0243"
 			(at 86.36 68.58 0)
 			(effects
@@
 			(project "arb"
 				(path "/866ef9be-3b01-4288-a6e0-a2357aa17e50/15631b2d-3708-4ae8-a4e9-7f8a7b587733"
-					(reference "#PWR0231")
+					(reference "#PWR0243")
 					(unit 1)
 				)
@@
 		(dnp no)
 		(fields_autoplaced yes)
-		(property "Reference" "#PWR0246"
+		(property "Reference" "#PWR0258"
 			(at 228.6 74.93 0)
 			(effects
@@
 			(project "arb"
 				(path "/866ef9be-3b01-4288-a6e0-a2357aa17e50/15631b2d-3708-4ae8-a4e9-7f8a7b587733"
-					(reference "#PWR0246")
+					(reference "#PWR0258")
 					(unit 1)
 				)
@@
 		(dnp no)
 		(fields_autoplaced yes)
-		(property "Reference" "C96"
+		(property "Reference" "C101"
 			(at 234.95 105.4163 0)
 			(effects
@@
 			(project "arb"
 				(path "/866ef9be-3b01-4288-a6e0-a2357aa17e50/15631b2d-3708-4ae8-a4e9-7f8a7b587733"
-					(reference "C96")
+					(reference "C101")
 					(unit 1)
 				)
@@
 		(on_board yes)
 		(dnp no)
-		(property "Reference" "#PWR0244"
+		(property "Reference" "#PWR0256"
 			(at 224.79 109.22 0)
 			(effects
@@
 			(project "arb"
 				(path "/866ef9be-3b01-4288-a6e0-a2357aa17e50/15631b2d-3708-4ae8-a4e9-7f8a7b587733"
-					(reference "#PWR0244")
+					(reference "#PWR0256")
 					(unit 1)
 				)
@@
 		(on_board yes)
 		(dnp no)
-		(property "Reference" "#PWR0242"
+		(property "Reference" "#PWR0254"
 			(at 209.55 101.6 0)
 			(effects
@@
 			(project "arb"
 				(path "/866ef9be-3b01-4288-a6e0-a2357aa17e50/15631b2d-3708-4ae8-a4e9-7f8a7b587733"
-					(reference "#PWR0242")
+					(reference "#PWR0254")
 					(unit 1)
 				)
@@
 		(dnp no)
 		(fields_autoplaced yes)
-		(property "Reference" "#PWR0234"
+		(property "Reference" "#PWR0246"
 			(at 100.33 67.31 0)
 			(effects
@@
 			(project "arb"
 				(path "/866ef9be-3b01-4288-a6e0-a2357aa17e50/15631b2d-3708-4ae8-a4e9-7f8a7b587733"
-					(reference "#PWR0234")
+					(reference "#PWR0246")
 					(unit 1)
 				)
@@
 		(dnp no)
 		(fields_autoplaced yes)
-		(property "Reference" "#PWR0245"
+		(property "Reference" "#PWR0257"
 			(at 227.33 109.22 0)
 			(effects
@@
 			(project "arb"
 				(path "/866ef9be-3b01-4288-a6e0-a2357aa17e50/15631b2d-3708-4ae8-a4e9-7f8a7b587733"
-					(reference "#PWR0245")
+					(reference "#PWR0257")
 					(unit 1)
 				)
@@
 		(dnp no)
 		(fields_autoplaced yes)
-		(property "Reference" "C91"
+		(property "Reference" "C96"
 			(at 106.68 38.1063 0)
 			(effects
@@
 			(project "arb"
 				(path "/866ef9be-3b01-4288-a6e0-a2357aa17e50/15631b2d-3708-4ae8-a4e9-7f8a7b587733"
-					(reference "C91")
+					(reference "C96")
 					(unit 1)
 				)
@@
 		(dnp no)
 		(fields_autoplaced yes)
-		(property "Reference" "#PWR0230"
+		(property "Reference" "#PWR0242"
 			(at 68.58 137.16 0)
 			(effects
@@
 			(project "arb"
 				(path "/866ef9be-3b01-4288-a6e0-a2357aa17e50/15631b2d-3708-4ae8-a4e9-7f8a7b587733"
-					(reference "#PWR0230")
+					(reference "#PWR0242")
 					(unit 1)
 				)
@@
 		(dnp no)
 		(fields_autoplaced yes)
-		(property "Reference" "#PWR0235"
+		(property "Reference" "#PWR0247"
 			(at 100.33 107.95 0)
 			(effects
@@
 			(project "arb"
 				(path "/866ef9be-3b01-4288-a6e0-a2357aa17e50/15631b2d-3708-4ae8-a4e9-7f8a7b587733"
-					(reference "#PWR0235")
+					(reference "#PWR0247")
 					(unit 1)
 				)
@@
 		(dnp no)
 		(fields_autoplaced yes)
-		(property "Reference" "#PWR0247"
+		(property "Reference" "#PWR0259"
 			(at 232.41 115.57 0)
 			(effects
@@
 			(project "arb"
 				(path "/866ef9be-3b01-4288-a6e0-a2357aa17e50/15631b2d-3708-4ae8-a4e9-7f8a7b587733"
-					(reference "#PWR0247")
+					(reference "#PWR0259")
 					(unit 1)
 				)
@@
 		(dnp no)
 		(fields_autoplaced yes)
-		(property "Reference" "C94"
+		(property "Reference" "C99"
 			(at 107.95 132.0863 0)
 			(effects
@@
 			(project "arb"
 				(path "/866ef9be-3b01-4288-a6e0-a2357aa17e50/15631b2d-3708-4ae8-a4e9-7f8a7b587733"
-					(reference "C94")
+					(reference "C99")
 					(unit 1)
 				)
@@
 		(dnp no)
 		(fields_autoplaced yes)
-		(property "Reference" "#PWR0229"
+		(property "Reference" "#PWR0241"
 			(at 68.58 68.58 0)
 			(effects
@@
 			(project "arb"
 				(path "/866ef9be-3b01-4288-a6e0-a2357aa17e50/15631b2d-3708-4ae8-a4e9-7f8a7b587733"
-					(reference "#PWR0229")
+					(reference "#PWR0241")
 					(unit 1)
 				)
@@
 		(pin "5"
 		)
-		(pin "14"
+		(pin "12"
 		)
 		(pin "7"
@@
 		(dnp no)
 		(fields_autoplaced yes)
-		(property "Reference" "#PWR0236"
+		(property "Reference" "#PWR0248"
 			(at 100.33 135.89 0)
 			(effects
@@
 			(project "arb"
 				(path "/866ef9be-3b01-4288-a6e0-a2357aa17e50/15631b2d-3708-4ae8-a4e9-7f8a7b587733"
-					(reference "#PWR0236")
+					(reference "#PWR0248")
 					(unit 1)
 				)
@@
 		(dnp yes)
 		(fields_autoplaced yes)
-		(property "Reference" "C90"
+		(property "Reference" "C95"
 			(at 63.5063 107.95 90)
 			(effects
@@
 			(project "arb"
 				(path "/866ef9be-3b01-4288-a6e0-a2357aa17e50/15631b2d-3708-4ae8-a4e9-7f8a7b587733"
-					(reference "C90")
+					(reference "C95")
 					(unit 1)
 				)
@@
 		(dnp no)
 		(fields_autoplaced yes)
-		(property "Reference" "C95"
+		(property "Reference" "C100"
 			(at 231.14 64.7763 0)
 			(effects
@@
 			(project "arb"
 				(path "/866ef9be-3b01-4288-a6e0-a2357aa17e50/15631b2d-3708-4ae8-a4e9-7f8a7b587733"
-					(reference "C95")
+					(reference "C100")
 					(unit 1)
 				)
@@
 		(dnp no)
 		(fields_autoplaced yes)
-		(property "Reference" "#PWR0243"
+		(property "Reference" "#PWR0255"
 			(at 224.79 66.04 0)
 			(effects
@@
 			(project "arb"
 				(path "/866ef9be-3b01-4288-a6e0-a2357aa17e50/15631b2d-3708-4ae8-a4e9-7f8a7b587733"
-					(reference "#PWR0243")
+					(reference "#PWR0255")
 					(unit 1)
 				)
@@
 		(dnp no)
 		(fields_autoplaced yes)
-		(property "Reference" "#PWR0227"
+		(property "Reference" "#PWR0239"
 			(at 58.42 68.58 0)
 			(effects
@@
 			(project ""
 				(path "/866ef9be-3b01-4288-a6e0-a2357aa17e50/15631b2d-3708-4ae8-a4e9-7f8a7b587733"
-					(reference "#PWR0227")
+					(reference "#PWR0239")
 					(unit 1)
 				)
@@
 		(dnp no)
 		(fields_autoplaced yes)
-		(property "Reference" "#PWR0241"
+		(property "Reference" "#PWR0253"
 			(at 204.47 115.57 0)
 			(effects
@@
 			(project "arb"
 				(path "/866ef9be-3b01-4288-a6e0-a2357aa17e50/15631b2d-3708-4ae8-a4e9-7f8a7b587733"
-					(reference "#PWR0241")
+					(reference "#PWR0253")
 					(unit 1)
 				)
@@
 		(dnp no)
 		(fields_autoplaced yes)
-		(property "Reference" "#PWR0232"
+		(property "Reference" "#PWR0244"
 			(at 86.36 137.16 0)
 			(effects
@@
 			(project "arb"
 				(path "/866ef9be-3b01-4288-a6e0-a2357aa17e50/15631b2d-3708-4ae8-a4e9-7f8a7b587733"
-					(reference "#PWR0232")
+					(reference "#PWR0244")
 					(unit 1)
 				)
@@
 		(dnp no)
 		(fields_autoplaced yes)
-		(property "Reference" "C92"
+		(property "Reference" "C97"
 			(at 106.68 106.6863 0)
 			(effects
@@
 			(project "arb"
 				(path "/866ef9be-3b01-4288-a6e0-a2357aa17e50/15631b2d-3708-4ae8-a4e9-7f8a7b587733"
-					(reference "C92")
+					(reference "C97")
 					(unit 1)
 				)
@@
 		(dnp no)
 		(fields_autoplaced yes)
-		(property "Reference" "C93"
+		(property "Reference" "C98"
 			(at 107.95 63.5063 0)
 			(effects
@@
 			(project "arb"
 				(path "/866ef9be-3b01-4288-a6e0-a2357aa17e50/15631b2d-3708-4ae8-a4e9-7f8a7b587733"
-					(reference "C93")
+					(reference "C98")
 					(unit 1)
 				)
@@
 		(dnp no)
 		(fields_autoplaced yes)
-		(property "Reference" "#PWR0238"
+		(property "Reference" "#PWR0250"
 			(at 104.14 116.84 0)
 			(effects
@@
 			(project "arb"
 				(path "/866ef9be-3b01-4288-a6e0-a2357aa17e50/15631b2d-3708-4ae8-a4e9-7f8a7b587733"
-					(reference "#PWR0238")
+					(reference "#PWR0250")
 					(unit 1)
 				)
@@
 		(dnp no)
 		(fields_autoplaced yes)
-		(property "Reference" "#PWR0240"
+		(property "Reference" "#PWR0252"
 			(at 105.41 142.24 0)
 			(effects
@@
 			(project "arb"
 				(path "/866ef9be-3b01-4288-a6e0-a2357aa17e50/15631b2d-3708-4ae8-a4e9-7f8a7b587733"
-					(reference "#PWR0240")
+					(reference "#PWR0252")
 					(unit 1)
 				)
@@
 		(dnp no)
 		(fields_autoplaced yes)
-		(property "Reference" "#PWR0228"
+		(property "Reference" "#PWR0240"
 			(at 58.42 137.16 0)
 			(effects
@@
 			(project "arb"
 				(path "/866ef9be-3b01-4288-a6e0-a2357aa17e50/15631b2d-3708-4ae8-a4e9-7f8a7b587733"
-					(reference "#PWR0228")
+					(reference "#PWR0240")
 					(unit 1)
 				)
@@
 		(dnp no)
 		(fields_autoplaced yes)
-		(property "Reference" "#PWR0237"
+		(property "Reference" "#PWR0249"
 			(at 104.14 48.26 0)
 			(effects
@@
 			(project "arb"
 				(path "/866ef9be-3b01-4288-a6e0-a2357aa17e50/15631b2d-3708-4ae8-a4e9-7f8a7b587733"
-					(reference "#PWR0237")
+					(reference "#PWR0249")
 					(unit 1)
 				)
@@
 		(dnp no)
 		(fields_autoplaced yes)
-		(property "Reference" "#PWR0239"
+		(property "Reference" "#PWR0251"
 			(at 105.41 73.66 0)
 			(effects
@@
 			(project "arb"
 				(path "/866ef9be-3b01-4288-a6e0-a2357aa17e50/15631b2d-3708-4ae8-a4e9-7f8a7b587733"
-					(reference "#PWR0239")
+					(reference "#PWR0251")
 					(unit 1)
 				)

Commit message: FEAT: Changed Inductor to higher current. Continued layout. Assigned some Netclasses.
Parts:
- renumbered C99 to C100, C100 to C101, C101 to C102, C94 to C95, C95 to C96, C96 to C97, C97 to C98, C98 to C99
Changed lines of the file:
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@@
 		(on_board yes)
 		(dnp no)
-		(property "Reference" "#PWR0245"
+		(property "Reference" "#PWR0247"
 			(at 100.33 39.37 0)
 			(effects
@@
 			(project "arb"
 				(path "/866ef9be-3b01-4288-a6e0-a2357aa17e50/15631b2d-3708-4ae8-a4e9-7f8a7b587733"
-					(reference "#PWR0245")
+					(reference "#PWR0247")
 					(unit 1)
 				)
@@
 		(dnp yes)
 		(fields_autoplaced yes)
-		(property "Reference" "C94"
+		(property "Reference" "C95"
 			(at 63.5063 39.37 90)
 			(effects
@@
 			(project ""
 				(path "/866ef9be-3b01-4288-a6e0-a2357aa17e50/15631b2d-3708-4ae8-a4e9-7f8a7b587733"
-					(reference "C94")
+					(reference "C95")
 					(unit 1)
 				)
@@
 		(dnp no)
 		(fields_autoplaced yes)
-		(property "Reference" "#PWR0243"
+		(property "Reference" "#PWR0245"
 			(at 86.36 68.58 0)
 			(effects
@@
 			(project "arb"
 				(path "/866ef9be-3b01-4288-a6e0-a2357aa17e50/15631b2d-3708-4ae8-a4e9-7f8a7b587733"
-					(reference "#PWR0243")
+					(reference "#PWR0245")
 					(unit 1)
 				)
@@
 		(dnp no)
 		(fields_autoplaced yes)
-		(property "Reference" "#PWR0258"
+		(property "Reference" "#PWR0260"
 			(at 228.6 74.93 0)
 			(effects
@@
 			(project "arb"
 				(path "/866ef9be-3b01-4288-a6e0-a2357aa17e50/15631b2d-3708-4ae8-a4e9-7f8a7b587733"
-					(reference "#PWR0258")
+					(reference "#PWR0260")
 					(unit 1)
 				)
@@
 		(dnp no)
 		(fields_autoplaced yes)
-		(property "Reference" "C101"
+		(property "Reference" "C102"
 			(at 234.95 105.4163 0)
 			(effects
@@
 			(project "arb"
 				(path "/866ef9be-3b01-4288-a6e0-a2357aa17e50/15631b2d-3708-4ae8-a4e9-7f8a7b587733"
-					(reference "C101")
+					(reference "C102")
 					(unit 1)
 				)
@@
 		(on_board yes)
 		(dnp no)
-		(property "Reference" "#PWR0256"
+		(property "Reference" "#PWR0258"
 			(at 224.79 109.22 0)
 			(effects
@@
 			(project "arb"
 				(path "/866ef9be-3b01-4288-a6e0-a2357aa17e50/15631b2d-3708-4ae8-a4e9-7f8a7b587733"
-					(reference "#PWR0256")
+					(reference "#PWR0258")
 					(unit 1)
 				)
@@
 		(on_board yes)
 		(dnp no)
-		(property "Reference" "#PWR0254"
+		(property "Reference" "#PWR0256"
 			(at 209.55 101.6 0)
 			(effects
@@
 			(project "arb"
 				(path "/866ef9be-3b01-4288-a6e0-a2357aa17e50/15631b2d-3708-4ae8-a4e9-7f8a7b587733"
-					(reference "#PWR0254")
+					(reference "#PWR0256")
 					(unit 1)
 				)
@@
 		(dnp no)
 		(fields_autoplaced yes)
-		(property "Reference" "#PWR0246"
+		(property "Reference" "#PWR0248"
 			(at 100.33 67.31 0)
 			(effects
@@
 			(project "arb"
 				(path "/866ef9be-3b01-4288-a6e0-a2357aa17e50/15631b2d-3708-4ae8-a4e9-7f8a7b587733"
-					(reference "#PWR0246")
+					(reference "#PWR0248")
 					(unit 1)
 				)
@@
 		(dnp no)
 		(fields_autoplaced yes)
-		(property "Reference" "#PWR0257"
+		(property "Reference" "#PWR0259"
 			(at 227.33 109.22 0)
 			(effects
@@
 			(project "arb"
 				(path "/866ef9be-3b01-4288-a6e0-a2357aa17e50/15631b2d-3708-4ae8-a4e9-7f8a7b587733"
-					(reference "#PWR0257")
+					(reference "#PWR0259")
 					(unit 1)
 				)
@@
 		(dnp no)
 		(fields_autoplaced yes)
-		(property "Reference" "C96"
+		(property "Reference" "C97"
 			(at 106.68 38.1063 0)
 			(effects
@@
 			(project "arb"
 				(path "/866ef9be-3b01-4288-a6e0-a2357aa17e50/15631b2d-3708-4ae8-a4e9-7f8a7b587733"
-					(reference "C96")
+					(reference "C97")
 					(unit 1)
 				)
@@
 		(dnp no)
 		(fields_autoplaced yes)
-		(property "Reference" "#PWR0242"
+		(property "Reference" "#PWR0244"
 			(at 68.58 137.16 0)
 			(effects
@@
 			(project "arb"
 				(path "/866ef9be-3b01-4288-a6e0-a2357aa17e50/15631b2d-3708-4ae8-a4e9-7f8a7b587733"
-					(reference "#PWR0242")
+					(reference "#PWR0244")
 					(unit 1)
 				)
@@
 		(dnp no)
 		(fields_autoplaced yes)
-		(property "Reference" "#PWR0247"
+		(property "Reference" "#PWR0249"
 			(at 100.33 107.95 0)
 			(effects
@@
 			(project "arb"
 				(path "/866ef9be-3b01-4288-a6e0-a2357aa17e50/15631b2d-3708-4ae8-a4e9-7f8a7b587733"
-					(reference "#PWR0247")
+					(reference "#PWR0249")
 					(unit 1)
 				)
@@
 		(dnp no)
 		(fields_autoplaced yes)
-		(property "Reference" "#PWR0259"
+		(property "Reference" "#PWR0261"
 			(at 232.41 115.57 0)
 			(effects
@@
 			(project "arb"
 				(path "/866ef9be-3b01-4288-a6e0-a2357aa17e50/15631b2d-3708-4ae8-a4e9-7f8a7b587733"
-					(reference "#PWR0259")
+					(reference "#PWR0261")
 					(unit 1)
 				)
@@
 		(dnp no)
 		(fields_autoplaced yes)
-		(property "Reference" "C99"
+		(property "Reference" "C100"
 			(at 107.95 132.0863 0)
 			(effects
@@
 			(project "arb"
 				(path "/866ef9be-3b01-4288-a6e0-a2357aa17e50/15631b2d-3708-4ae8-a4e9-7f8a7b587733"
-					(reference "C99")
+					(reference "C100")
 					(unit 1)
 				)
@@
 		(dnp no)
 		(fields_autoplaced yes)
-		(property "Reference" "#PWR0241"
+		(property "Reference" "#PWR0243"
 			(at 68.58 68.58 0)
 			(effects
@@
 			(project "arb"
 				(path "/866ef9be-3b01-4288-a6e0-a2357aa17e50/15631b2d-3708-4ae8-a4e9-7f8a7b587733"
-					(reference "#PWR0241")
+					(reference "#PWR0243")
 					(unit 1)
 				)
@@
 		(dnp no)
 		(fields_autoplaced yes)
-		(property "Reference" "#PWR0248"
+		(property "Reference" "#PWR0250"
 			(at 100.33 135.89 0)
 			(effects
@@
 			(project "arb"
 				(path "/866ef9be-3b01-4288-a6e0-a2357aa17e50/15631b2d-3708-4ae8-a4e9-7f8a7b587733"
-					(reference "#PWR0248")
+					(reference "#PWR0250")
 					(unit 1)
 				)
@@
 		(dnp yes)
 		(fields_autoplaced yes)
-		(property "Reference" "C95"
+		(property "Reference" "C96"
 			(at 63.5063 107.95 90)
 			(effects
@@
 			(project "arb"
 				(path "/866ef9be-3b01-4288-a6e0-a2357aa17e50/15631b2d-3708-4ae8-a4e9-7f8a7b587733"
-					(reference "C95")
+					(reference "C96")
 					(unit 1)
 				)
@@
 		(dnp no)
 		(fields_autoplaced yes)
-		(property "Reference" "C100"
+		(property "Reference" "C101"
 			(at 231.14 64.7763 0)
 			(effects
@@
 			(project "arb"
 				(path "/866ef9be-3b01-4288-a6e0-a2357aa17e50/15631b2d-3708-4ae8-a4e9-7f8a7b587733"
-					(reference "C100")
+					(reference "C101")
 					(unit 1)
 				)
@@
 		(dnp no)
 		(fields_autoplaced yes)
-		(property "Reference" "#PWR0255"
+		(property "Reference" "#PWR0257"
 			(at 224.79 66.04 0)
 			(effects
@@
 			(project "arb"
 				(path "/866ef9be-3b01-4288-a6e0-a2357aa17e50/15631b2d-3708-4ae8-a4e9-7f8a7b587733"
-					(reference "#PWR0255")
+					(reference "#PWR0257")
 					(unit 1)
 				)
@@
 		(dnp no)
 		(fields_autoplaced yes)
-		(property "Reference" "#PWR0239"
+		(property "Reference" "#PWR0241"
 			(at 58.42 68.58 0)
 			(effects
@@
 			(project ""
 				(path "/866ef9be-3b01-4288-a6e0-a2357aa17e50/15631b2d-3708-4ae8-a4e9-7f8a7b587733"
-					(reference "#PWR0239")
+					(reference "#PWR0241")
 					(unit 1)
 				)
@@
 		(dnp no)
 		(fields_autoplaced yes)
-		(property "Reference" "#PWR0253"
+		(property "Reference" "#PWR0255"
 			(at 204.47 115.57 0)
 			(effects
@@
 			(project "arb"
 				(path "/866ef9be-3b01-4288-a6e0-a2357aa17e50/15631b2d-3708-4ae8-a4e9-7f8a7b587733"
-					(reference "#PWR0253")
+					(reference "#PWR0255")
 					(unit 1)
 				)
@@
 		(dnp no)
 		(fields_autoplaced yes)
-		(property "Reference" "#PWR0244"
+		(property "Reference" "#PWR0246"
 			(at 86.36 137.16 0)
 			(effects
@@
 			(project "arb"
 				(path "/866ef9be-3b01-4288-a6e0-a2357aa17e50/15631b2d-3708-4ae8-a4e9-7f8a7b587733"
-					(reference "#PWR0244")
+					(reference "#PWR0246")
 					(unit 1)
 				)
@@
 		(dnp no)
 		(fields_autoplaced yes)
-		(property "Reference" "C97"
+		(property "Reference" "C98"
 			(at 106.68 106.6863 0)
 			(effects
@@
 			(project "arb"
 				(path "/866ef9be-3b01-4288-a6e0-a2357aa17e50/15631b2d-3708-4ae8-a4e9-7f8a7b587733"
-					(reference "C97")
+					(reference "C98")
 					(unit 1)
 				)
@@
 		(dnp no)
 		(fields_autoplaced yes)
-		(property "Reference" "C98"
+		(property "Reference" "C99"
 			(at 107.95 63.5063 0)
 			(effects
@@
 			(project "arb"
 				(path "/866ef9be-3b01-4288-a6e0-a2357aa17e50/15631b2d-3708-4ae8-a4e9-7f8a7b587733"
-					(reference "C98")
+					(reference "C99")
 					(unit 1)
 				)
@@
 		(dnp no)
 		(fields_autoplaced yes)
-		(property "Reference" "#PWR0250"
+		(property "Reference" "#PWR0252"
 			(at 104.14 116.84 0)
 			(effects
@@
 			(project "arb"
 				(path "/866ef9be-3b01-4288-a6e0-a2357aa17e50/15631b2d-3708-4ae8-a4e9-7f8a7b587733"
-					(reference "#PWR0250")
+					(reference "#PWR0252")
 					(unit 1)
 				)
@@
 		(dnp no)
 		(fields_autoplaced yes)
-		(property "Reference" "#PWR0252"
+		(property "Reference" "#PWR0254"
 			(at 105.41 142.24 0)
 			(effects
@@
 			(project "arb"
 				(path "/866ef9be-3b01-4288-a6e0-a2357aa17e50/15631b2d-3708-4ae8-a4e9-7f8a7b587733"
-					(reference "#PWR0252")
+					(reference "#PWR0254")
 					(unit 1)
 				)
@@
 		(dnp no)
 		(fields_autoplaced yes)
-		(property "Reference" "#PWR0240"
+		(property "Reference" "#PWR0242"
 			(at 58.42 137.16 0)
 			(effects
@@
 			(project "arb"
 				(path "/866ef9be-3b01-4288-a6e0-a2357aa17e50/15631b2d-3708-4ae8-a4e9-7f8a7b587733"
-					(reference "#PWR0240")
+					(reference "#PWR0242")
 					(unit 1)
 				)
@@
 		(dnp no)
 		(fields_autoplaced yes)
-		(property "Reference" "#PWR0249"
+		(property "Reference" "#PWR0251"
 			(at 104.14 48.26 0)
 			(effects
@@
 			(project "arb"
 				(path "/866ef9be-3b01-4288-a6e0-a2357aa17e50/15631b2d-3708-4ae8-a4e9-7f8a7b587733"
-					(reference "#PWR0249")
+					(reference "#PWR0251")
 					(unit 1)
 				)
@@
 		(dnp no)
 		(fields_autoplaced yes)
-		(property "Reference" "#PWR0251"
+		(property "Reference" "#PWR0253"
 			(at 105.41 73.66 0)
 			(effects
@@
 			(project "arb"
 				(path "/866ef9be-3b01-4288-a6e0-a2357aa17e50/15631b2d-3708-4ae8-a4e9-7f8a7b587733"
-					(reference "#PWR0251")
+					(reference "#PWR0253")
 					(unit 1)
 				)
