File: 1_hw/03_pcb/power.kicad_sch (KiCad schematic)
At the start: 61 parts, among them U1 TLV70333DBV, U10 TPS65131RGE, U11 TPD2E001DRL, U4 TLV76133DCY, U5 TLV70333DBV, U6 LM3880MF-1AA, U8 TLV70312DBV, U9 TLV70325DBV

Commit message: FEAT: Assigned Reference Designators; Assigned Passives Part Numbers & Footprints (0603); Assigned LCSC P/Ns.
Parts:
- C1, C2: footprint (none) -> Capacitor_SMD:C_0603_1608Metric; LCSC (none) -> C15849; Part Number (none) -> CL10A105KB8NNNC
- C10: renamed from C46; footprint (none) -> Capacitor_SMD:C_0603_1608Metric; LCSC (none) -> C23630; Part Number (none) -> CL10A225KO8NNNC
- C11: renamed from C47; footprint (none) -> Capacitor_SMD:C_0603_1608Metric; LCSC (none) -> C15849; Part Number (none) -> CL10A105KB8NNNC
- C12: renamed from C48; footprint (none) -> Capacitor_SMD:C_0603_1608Metric; LCSC (none) -> C15849; Part Number (none) -> CL10A105KB8NNNC
- C13: renamed from C49; footprint (none) -> Capacitor_SMD:C_0603_1608Metric; LCSC (none) -> C23630; Part Number (none) -> CL10A225KO8NNNC
- C14: renamed from C50; footprint (none) -> Capacitor_SMD:C_0603_1608Metric; LCSC (none) -> C23630; Part Number (none) -> CL10A225KO8NNNC
- C15: renamed from C51; footprint (none) -> Capacitor_SMD:C_0603_1608Metric; LCSC (none) -> C1705; Part Number (none) -> CL10A475KP8NNNC
- C16: renamed from C52; value 0.1u -> 100n; footprint (none) -> Capacitor_SMD:C_0603_1608Metric; LCSC (none) -> C24452; Part Number (none) -> CL10B104JB8NNNC
- C17: renamed from C53; value 0.01u -> 10n; footprint (none) -> Capacitor_SMD:C_0603_1608Metric; LCSC (none) -> C1589; Part Number (none) -> CL10B103KB8NNNC
- C18: renamed from C54; value 4700p -> 4.7n; footprint (none) -> Capacitor_SMD:C_0603_1608Metric; LCSC (none) -> C106218; Part Number (none) -> CC0603KRX7R9BB472
- C19: renamed from C55; footprint (none) -> Capacitor_SMD:C_0603_1608Metric; LCSC (none) -> C519114; Part Number (none) -> CC0603BRNPO9BN6R8
- C20: renamed from C56; value 0.22u -> 220n; footprint (none) -> Capacitor_SMD:C_0603_1608Metric; LCSC (none) -> C64705; Part Number (none) -> CL10B224KB8NNNC
- C21: renamed from C57; footprint (none) -> Capacitor_SMD:C_0603_1608Metric; LCSC (none) -> C519114; Part Number (none) -> CC0603BRNPO9BN6R8
- C22: renamed from C58; footprint (none) -> Capacitor_SMD:C_0603_1608Metric; LCSC (none) -> C1705; Part Number (none) -> CL10A475KP8NNNC
- C23: renamed from C59; footprint (none) -> Capacitor_SMD:C_0603_1608Metric; LCSC (none) -> C1705; Part Number (none) -> CL10A475KP8NNNC
- C24: renamed from C60; footprint (none) -> Capacitor_SMD:C_0603_1608Metric; LCSC (none) -> C1705; Part Number (none) -> CL10A475KP8NNNC
- C25: renamed from C61; footprint (none) -> Capacitor_SMD:C_0603_1608Metric; LCSC (none) -> C1705; Part Number (none) -> CL10A475KP8NNNC
- C26: renamed from C62; footprint (none) -> Capacitor_SMD:C_0603_1608Metric; LCSC (none) -> C1705; Part Number (none) -> CL10A475KP8NNNC
- C27: renamed from C63; footprint (none) -> Capacitor_SMD:C_0603_1608Metric; LCSC (none) -> C1705; Part Number (none) -> CL10A475KP8NNNC
- C28: renamed from C64; LCSC (none) -> C24452; PN CL10B104JB8NNNC -> (none); Part Number (none) -> CL10B104JB8NNNC
- C29: renamed from C65; footprint (none) -> Capacitor_SMD:C_0603_1608Metric; LCSC (none) -> C1705; Part Number (none) -> CL10A475KP8NNNC
- C3: renamed from C39; footprint (none) -> Capacitor_SMD:C_0603_1608Metric; LCSC (none) -> C15849; Part Number (none) -> CL10A105KB8NNNC
- C30: renamed from C66; footprint (none) -> Capacitor_SMD:C_0603_1608Metric; LCSC (none) -> C1705; Part Number (none) -> CL10A475KP8NNNC
- C31: renamed from C67; footprint (none) -> Capacitor_SMD:C_0603_1608Metric; LCSC (none) -> C24452; Part Number (none) -> CL10B104JB8NNNC
- C32: renamed from C68; footprint (none) -> Capacitor_SMD:C_0603_1608Metric; LCSC (none) -> C24452; Part Number (none) -> CL10B104JB8NNNC
- C4: renamed from C40; footprint (none) -> Capacitor_SMD:C_0603_1608Metric; LCSC (none) -> C19702; Part Number (none) -> CL10A106KP8NNNC
- C5: renamed from C41; footprint (none) -> Capacitor_SMD:C_0603_1608Metric; LCSC (none) -> C1705; Part Number (none) -> CL10A475KP8NNNC
- C6: renamed from C42; LCSC (none) -> C24452; PN CL10B104JB8NNNC -> (none); Part Number (none) -> CL10B104JB8NNNC
- C7: renamed from C43; footprint (none) -> Capacitor_SMD:C_0603_1608Metric; LCSC (none) -> C15849; Part Number (none) -> CL10A105KB8NNNC
- C8: renamed from C44; footprint (none) -> Capacitor_SMD:C_0603_1608Metric; LCSC (none) -> C23630; Part Number (none) -> CL10A225KO8NNNC
- C9: renamed from C45; footprint (none) -> Capacitor_SMD:C_0603_1608Metric; LCSC (none) -> C23630; Part Number (none) -> CL10A225KO8NNNC
- D1: renamed from D3; footprint BRZK_TBD -> (none); LCSC (none) -> C152484
- D2: renamed from D4; footprint BRZK_TBD -> (none); LCSC (none) -> C152484
- L1: renamed from L3; footprint (none) -> Inductor_SMD:L_0603_1608Metric; LCSC (none) -> C114862; Part Number (none) -> LQM18PN4R7MFRL
- L2: renamed from L4; footprint (none) -> Inductor_SMD:L_0603_1608Metric; LCSC (none) -> C114862; Part Number (none) -> LQM18PN4R7MFRL
- R1: renamed from R2; LCSC (none) -> C25804; PN CR-03FC7---10K -> (none); Part Number (none) -> 0603WAF1002T5E
- R10: renamed from R20; footprint (none) -> Resistor_SMD:R_0603_1608Metric; LCSC (none) -> C15402; Part Number (none) -> 0603WAJ0000T5E
- R11: renamed from R21; footprint (none) -> Resistor_SMD:R_0603_1608Metric; LCSC (none) -> C15402; Part Number (none) -> 0603WAJ0000T5E
- R12: renamed from R22; value 104.8k -> 104k; footprint (none) -> Resistor_SMD:R_0603_1608Metric; LCSC (none) -> C862849; Part Number (none) -> RT0603DRE07104KL
- R13: renamed from R23; footprint (none) -> Resistor_SMD:R_0603_1608Metric; LCSC (none) -> C245931; Part Number (none) -> RC0603FR-071M3L
- R14: renamed from R24; footprint (none) -> Resistor_SMD:R_0603_1608Metric; LCSC (none) -> C15402; Part Number (none) -> 0603WAJ0000T5E
- R15: renamed from R25; footprint (none) -> Resistor_SMD:R_0603_1608Metric; LCSC (none) -> C15402; Part Number (none) -> 0603WAJ0000T5E
- R16: renamed from R26; LCSC (none) -> C15402; PN 0603WAJ0000T5E -> (none); Part Number (none) -> 0603WAJ0000T5E
- R17: renamed from R27; LCSC (none) -> C15402; PN 0603WAJ0000T5E -> (none); Part Number (none) -> 0603WAJ0000T5E
- R2: renamed from R3; LCSC (none) -> C25804; PN CR-03FC7---10K -> (none); Part Number (none) -> 0603WAF1002T5E
- R3: renamed from R4; LCSC (none) -> C25804; PN CR-03FC7---10K -> (none); Part Number (none) -> 0603WAF1002T5E
- R4: renamed from R15; footprint (none) -> Resistor_SMD:R_0603_1608Metric; LCSC (none) -> C25805; Part Number (none) -> 0603WAF1103T5E
- R5: renamed from R?; footprint (none) -> Resistor_SMD:R_0603_1608Metric; LCSC (none) -> C22935; Part Number (none) -> 0603WAF1004T5E
- R6: renamed from R16; footprint (none) -> Resistor_SMD:R_0603_1608Metric; LCSC (none) -> C15402; Part Number (none) -> 0603WAJ0000T5E
- R7: renamed from R17; footprint (none) -> Resistor_SMD:R_0603_1608Metric; LCSC (none) -> C15402; Part Number (none) -> 0603WAJ0000T5E
- R8: renamed from R18; footprint (none) -> Resistor_SMD:R_0603_1608Metric; LCSC (none) -> C48922; Part Number (none) -> 0603WAF9763T5E
- R9: renamed from R19; value 85.8k -> 84.5k; footprint (none) -> Resistor_SMD:R_0603_1608Metric; LCSC (none) -> C23118; Part Number (none) -> 0603WAF8452T5E
- U1: LCSC (none) -> C2871194
- U2: renamed from U4; LCSC (none) -> C7527500
- U3: renamed from U5; LCSC (none) -> C2871194
- U4: renamed from U6; LCSC (none) -> C486059
- U5: renamed from U8; LCSC (none) -> C2861352
- U6: renamed from U9; LCSC (none) -> C2877882
- U7: renamed from U10; LCSC (none) -> C87663; Part Number TPS65131RGE -> TPS65131RGER
- U8: renamed from U11; LCSC (none) -> C150526

Commit message: FEAT: Added MCU Flash. Finished creating & assigning footprints. Ran ERC & cleared out issues. Ready for Layout.
Parts:
- added D1: LED, LED_SMD:LED_1206_3216Metric, symbol Device:LED
- added R4: 499, Resistor_SMD:R_0603_1608Metric, symbol Device:R_Small_US
- D2: renamed from D1; footprint (none) -> BRZK_DIODE:D_SMP_DO-216AA
- D3: renamed from D2; footprint (none) -> BRZK_DIODE:D_SMP_DO-216AA
- U7: Part Number TPS65131RGER -> TPS65131RGE
- renumbered R9 to R10, R10 to R11, R11 to R12, R12 to R13, R13 to R14, R14 to R15, R15 to R16, R16 to R17, R17 to R18, R4 to R5, R5 to R6, R6 to R7, R7 to R8, R8 to R9
Connections:
- net 5P0V: now also R4.2
- net GND: now also D1.1 (K)
- new net: D1.2 (A), R4.1
Other:
- note added: "POWER LED"

Commit message: MINOR: Added Board Rules & Constraints.
Parts:
- U7: footprint Package_DFN_QFN:VQFN-24-1EP_4x4mm_P0.5mm_EP2.45x2.45mm_ThermalVias -> Package_DFN_QFN:VQFN-24-1EP_4x4mm_P0.5mm_EP2.45x2.45mm
Changed lines of the file:
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@@
 			)
 		)
-		(property "Footprint" "Package_DFN_QFN:VQFN-24-1EP_4x4mm_P0.5mm_EP2.45x2.45mm_ThermalVias"
+		(property "Footprint" "Package_DFN_QFN:VQFN-24-1EP_4x4mm_P0.5mm_EP2.45x2.45mm"
 			(at 158.75 132.08 0)
 			(effects

Commit message: FEAT: Changed Inductor to higher current. Continued layout. Assigned some Netclasses.
Parts:
- L1: footprint Inductor_SMD:L_0603_1608Metric -> BRZK_INDUCTOR:L_SMD_L2.5_W2.0_Metric; LCSC C114862 -> C5832360; Part Number LQM18PN4R7MFRL -> FTC252010S4R7MBCA
Changed lines of the file:
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@@
 			)
 		)
-		(property "Footprint" "Inductor_SMD:L_0603_1608Metric"
+		(property "Footprint" "BRZK_INDUCTOR:L_SMD_L2.5_W2.0_Metric"
 			(at 138.43 116.84 0)
 			(effects
@@
 			)
 		)
-		(property "LCSC" "C114862"
+		(property "LCSC" "     C5832360"
 			(at 138.43 116.84 0)
 			(effects
@@
 			)
 		)
-		(property "Part Number" "LQM18PN4R7MFRL"
+		(property "Part Number" "FTC252010S4R7MBCA"
 			(at 138.43 116.84 0)
 			(effects
