File: 1_hw/03_pcb/microprocessor.kicad_sch (KiCad schematic)
At the start: 29 parts, among them SW1 TS-1187A-B-A-B, SW2 SS-12D02-VG4, SW3 SS-12D02-VG4, U11 STM32F446ZETx, Y1 32.768k

Commit message: MINOR: Layout, working on SPI / QSPI. Currently mixed up.
Connections:
- net 3P3V_A: now also U11.6 (VBAT); no longer U11.33 (VDDA)
- net 3P3V_D: now also U11.33 (VDDA), U11.41 (PA5); no longer U11.32 (VREF+), U11.6 (VBAT), U11.95 (VDDUSB)
- net ANALOG_CAL-ADC_AMUX2_MCU: no longer U11.42 (PA6)
- net ANALOG_DAC1_MCU_AMUX1: no longer U11.40 (PA4)
- net ANALOG_DAC2_MCU_AMUX3: now also U11.32 (VREF+); no longer U11.41 (PA5)
- net CLK_10MHZ_DIST_MCU_3P3: now also U11.43 (PA7); no longer U11.23 (PH0)
- net GND: now also U11.82 (PD13), U11.85 (PD14); no longer U11.107 (VSS), U11.120 (VSS), U11.130 (VSS), U11.16 (VSS), U11.31 (VSSA), U11.38 (VSS), U11.51 (VSS), U11.61 (VSS), U11.83 (VSS), U11.94 (VSS)
- net GPIO_100M-EN_MCU_100M-OSC_3P3: now also U11.122 (PD6); no longer U11.66 (PE13)
- net GPIO_AMP-PD_MCU_AMP2_3P3: now also U11.102 (PA10); no longer U11.56 (PG0)
- net GPIO_BOOT0_SW_MCU_3P3_L: now also U11.37 (PA3); no longer U11.138 (BOOT0)
- net GPIO_BOOT1_SW_MCU_3P3_L: now also U11.124 (PG9); no longer U11.48 (PB2)
- net GPIO_CFG_DONE_FPGA_MCU_3P3: now also U11.114 (PD0); no longer U11.58 (PE7)
- net GPIO_CLK_EN_MCU_FPGA_3P3: now also U11.116 (PD2); no longer U11.60 (PE9)
- net GPIO_D0_MCU_DDS_3P3: now also U11.58 (PE7); no longer U11.114 (PD0)
- net GPIO_D1_MCU_DDS_3P3: now also U11.59 (PE8); no longer U11.115 (PD1)
- net GPIO_D2_MCU_DDS_3P3: now also U11.60 (PE9); no longer U11.116 (PD2)
- net GPIO_D3_MCU_DDS_3P3: now also U11.63 (PE10); no longer U11.117 (PD3)
- net GPIO_D4_MCU_DDS_3P3: now also U11.64 (PE11); no longer U11.118 (PD4)
- net GPIO_D5_MCU_DDS_3P3: now also U11.65 (PE12); no longer U11.119 (PD5)
- net GPIO_D6_MCU_DDS_3P3: now also U11.66 (PE13); no longer U11.122 (PD6)
- net GPIO_D7_MCU_DDS_3P3: now also U11.67 (PE14); no longer U11.123 (PD7)
- net GPIO_EN_MCU_AMUX1_3P3: now also U11.69 (PB10); no longer U11.10 (PF0)
- net GPIO_EN_MCU_AMUX2_3P3: now also U11.118 (PD4); no longer U11.64 (PE11)
- net GPIO_EN_MCU_AMUX3_3P3: now also U11.105 (PA13); no longer U11.88 (PG3)
- net GPIO_FPGARST_MCU_FPGA_3P3_L: now also U11.115 (PD1); no longer U11.59 (PE8)
- net GPIO_FQ-UD_MCU_DDS_3P3: no longer U11.78 (PD9)
- net GPIO_RST_MCU_3P3_L: now also U11.34 (PA0); no longer U11.25 (NRST)
- net GPIO_RST_MCU_DDS_3P3: now also U11.68 (PE15); no longer U11.77 (PD8)
- net GPIO_SEL0_MCU_AMUX1_3P3: now also U11.70 (PB11); no longer U11.11 (PF1)
- net GPIO_SEL0_MCU_AMUX3_3P3: now also U11.110 (PA15); no longer U11.90 (PG5)
- net GPIO_SEL1_MCU_AMUX1_3P3: now also U11.73 (PB12); no longer U11.12 (PF2)
- net GPIO_SEL1_MCU_AMUX3_3P3: now also U11.109 (PA14); no longer U11.89 (PG4)
- net GPIO_SEL_MCU_AMUX2_3P3: now also U11.119 (PD5); no longer U11.65 (PE12)
- net GPIO_SW-SEL_MCU_CLKMUX_3P3: now also U11.123 (PD7); no longer U11.67 (PE14)
- net GPIO_W-CLK_MCU_DDS_3P3: now also U11.71 (VCAP_1); no longer U11.79 (PD10)
- net I2C_SCL_MCU_POT_3P3: now also U11.10 (PF0); no longer U11.69 (PB10)
- net I2C_SDA_MCU_POT_3P3: now also U11.11 (PF1); no longer U11.70 (PB11)
- net JTAG_MCU_TCK_3P3: now also U11.89 (PG4); no longer U11.109 (PA14)
- net JTAG_MCU_TDI_3P3: now also U11.90 (PG5); no longer U11.110 (PA15)
- net JTAG_MCU_TDO_3P3: now also U11.125 (PG10); no longer U11.133 (PB3)
- net JTAG_MCU_TMS_3P3: now also U11.88 (PG3); no longer U11.105 (PA13)
- net QSPI_IO0_MCU_FLASH_3P3: now also U11.27 (PC1); no longer U11.20 (PF8)
- net QSPI_IO1_MCU_FLASH_3P3: now also U11.28 (PC2); no longer U11.21 (PF9)
- net QSPI_IO2_MCU_FLASH_3P3: now also U11.113 (PC12); no longer U11.1 (PE2)
- net QSPI_IO3_MCU_FLASH_3P3: no longer U11.18 (PF6)
- net QSPI_NCS_MCU_FLASH_3P3: no longer U11.91 (PG6)
- net SPI_CS_MCU_FLASH_3P3_L: no longer U11.29 (PC3)
- net SPI_CS_MCU_FPGA_3P3_L: no longer U11.26 (PC0)
- net SPI_MISO_FPGA_MCU_3P3: now also U11.21 (PF9); no longer U11.28 (PC2)
- net SPI_MOSI_MCU_FPGA_3P3: now also U11.20 (PF8); no longer U11.27 (PC1)
- net SPI_SCLK_MCU_FPGA_3P3: now also U11.13 (PF3)
- net UART_FTDITX_MCURX_3P3: now also U11.138 (BOOT0); no longer U11.37 (PA3)
- net UART_MCUTX_FTDIRX_3P3: no longer U11.36 (PA2)
- net at C38.1: now also U11.79 (PD10); no longer U11.71 (VCAP_1)
- net at C43.1, Y1.1: now also U11.4 (PE5); no longer U11.9 (PC15)
- net at C45.1, Y1.2: now also U11.3 (PE4); no longer U11.8 (PC14)
- net at R31.2: now also U11.35 (PA1); no longer U11.143 (PDR_ON)
- net at U11.106 (VCAP_2): no longer C39.1
- net at U11.80 (PD11): now also C39.1
- new net: U11.107 (VSS), U11.120 (VSS), U11.130 (VSS), U11.16 (VSS), U11.38 (VSS), U11.51 (VSS), U11.61 (VSS), U11.83 (VSS), U11.94 (VSS)
- no-connect marks 66 -> 65
Changed lines of the file:
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@@
 	)
 	(no_connect
-		(at 111.76 105.41)
-	)
-	(no_connect
 		(at 111.76 130.81)
 	)
@@
 	(global_label "SPI_SCLK_MCU_FPGA_3P3"
 		(shape input)
-		(at 154.94 104.14 0)
+		(at 111.76 105.41 0)
 		(fields_autoplaced yes)
 		(effects
@@
 		)
 		(property "Intersheetrefs" "${INTERSHEET_REFS}"
-			(at 182.1156 104.14 0)
+			(at 138.9356 105.41 0)
 			(effects
 				(font
@@
 		)
 	)
-	(global_label "SPI_CS_MCU_FLASH_3P3_L"
-		(shape input)
-		(at 111.76 123.19 0)
-		(fields_autoplaced yes)
-		(effects
-			(font
-				(size 1.27 1.27)
-			)
-			(justify left)
-		)
-		(property "Intersheetrefs" "${INTERSHEET_REFS}"
-			(at 139.6613 123.19 0)
-			(effects
-				(font
-					(size 1.27 1.27)
-				)
-				(justify left)
-				(hide yes)
-			)
-		)
-	)
 	(global_label "GPIO_RST_MCU_3P3_L"
 		(shape input)
@@
 		)
 	)
+	(global_label "SPI_CS_MCU_FPGA_3P3_L"
+		(shape input)
+		(at 149.86 118.11 0)
+		(fields_autoplaced yes)
+		(effects
+			(font
+				(size 1.27 1.27)
+			)
+			(justify left)
+		)
+		(property "Intersheetrefs" "${INTERSHEET_REFS}"
+			(at 176.7332 118.11 0)
+			(effects
+				(font
+					(size 1.27 1.27)
+				)
+				(justify left)
+				(hide yes)
+			)
+		)
+	)
 	(global_label "GPIO_D7_MCU_DDS_3P3"
 		(shape input)
@@
 		)
 	)
-	(global_label "SPI_CS_MCU_FPGA_3P3_L"
+	(global_label "SPI_CS_MCU_FLASH_3P3_L"
 		(shape input)
-		(at 111.76 115.57 0)
+		(at 149.86 125.73 0)
 		(fields_autoplaced yes)
 		(effects
@@
 		)
 		(property "Intersheetrefs" "${INTERSHEET_REFS}"
-			(at 138.6332 115.57 0)
+			(at 177.7613 125.73 0)
 			(effects
 				(font
@@
 		(lib_id "BRZK_STM32:STM32F446ZETx")
 		(at 81.28 115.57 0)
+		(mirror y)
 		(unit 1)
 		(exclude_from_sim no)
@@
 		(dnp no)
 		(property "Reference" "U11"
-			(at 53.34 20.32 0)
+			(at 109.22 20.32 0)
 			(effects
 				(font
@@
 		)
 		(property "Value" "STM32F446ZETx"
-			(at 53.34 22.86 0)
+			(at 109.22 22.86 0)
 			(effects
 				(font
@@
 		)
 		(property "Footprint" "Package_QFP:LQFP-144_20x20mm_P0.5mm"
-			(at 55.88 201.93 0)
+			(at 106.68 201.93 0)
 			(effects
 				(font

Commit message: MINOR: Layout, working on SPI / QSPI. Fixed issues with Schematic.
Connections:
- net 3P3V_A: now also U11.33 (VDDA); no longer U11.6 (VBAT)
- net 3P3V_D: now also U11.32 (VREF+), U11.6 (VBAT), U11.95 (VDDUSB); no longer U11.33 (VDDA), U11.41 (PA5)
- net ANALOG_CAL-ADC_AMUX2_MCU: now also U11.42 (PA6)
- net ANALOG_DAC1_MCU_AMUX1: now also U11.40 (PA4)
- net ANALOG_DAC2_MCU_AMUX3: now also U11.41 (PA5); no longer U11.32 (VREF+)
- net CLK_10MHZ_DIST_MCU_3P3: now also U11.23 (PH0); no longer U11.43 (PA7)
- net GND: now also U11.107 (VSS), U11.120 (VSS), U11.130 (VSS), U11.16 (VSS), U11.31 (VSSA), U11.38 (VSS), U11.51 (VSS), U11.61 (VSS), U11.83 (VSS), U11.94 (VSS); no longer U11.82 (PD13), U11.85 (PD14)
- net GPIO_100M-EN_MCU_100M-OSC_3P3: now also U11.66 (PE13); no longer U11.122 (PD6)
- net GPIO_AMP-PD_MCU_AMP2_3P3: now also U11.56 (PG0); no longer U11.102 (PA10)
- net GPIO_BOOT0_SW_MCU_3P3_L: now also U11.138 (BOOT0); no longer U11.37 (PA3)
- net GPIO_BOOT1_SW_MCU_3P3_L: now also U11.48 (PB2); no longer U11.124 (PG9)
- net GPIO_CFG_DONE_FPGA_MCU_3P3: now also U11.58 (PE7); no longer U11.114 (PD0)
- net GPIO_CLK_EN_MCU_FPGA_3P3: now also U11.60 (PE9); no longer U11.116 (PD2)
- net GPIO_D0_MCU_DDS_3P3: now also U11.114 (PD0); no longer U11.58 (PE7)
- net GPIO_D1_MCU_DDS_3P3: now also U11.115 (PD1); no longer U11.59 (PE8)
- net GPIO_D2_MCU_DDS_3P3: now also U11.116 (PD2); no longer U11.60 (PE9)
- net GPIO_D3_MCU_DDS_3P3: now also U11.117 (PD3); no longer U11.63 (PE10)
- net GPIO_D4_MCU_DDS_3P3: now also U11.118 (PD4); no longer U11.64 (PE11)
- net GPIO_D5_MCU_DDS_3P3: now also U11.119 (PD5); no longer U11.65 (PE12)
- net GPIO_D6_MCU_DDS_3P3: now also U11.122 (PD6); no longer U11.66 (PE13)
- net GPIO_D7_MCU_DDS_3P3: now also U11.123 (PD7); no longer U11.67 (PE14)
- net GPIO_EN_MCU_AMUX1_3P3: now also U11.10 (PF0); no longer U11.69 (PB10)
- net GPIO_EN_MCU_AMUX2_3P3: now also U11.64 (PE11); no longer U11.118 (PD4)
- net GPIO_EN_MCU_AMUX3_3P3: now also U11.88 (PG3); no longer U11.105 (PA13)
- net GPIO_FPGARST_MCU_FPGA_3P3_L: now also U11.59 (PE8); no longer U11.115 (PD1)
- net GPIO_FQ-UD_MCU_DDS_3P3: now also U11.78 (PD9)
- net GPIO_RST_MCU_3P3_L: now also U11.25 (NRST); no longer U11.34 (PA0)
- net GPIO_RST_MCU_DDS_3P3: now also U11.77 (PD8); no longer U11.68 (PE15)
- net GPIO_SEL0_MCU_AMUX1_3P3: now also U11.11 (PF1); no longer U11.70 (PB11)
- net GPIO_SEL0_MCU_AMUX3_3P3: now also U11.90 (PG5); no longer U11.110 (PA15)
- net GPIO_SEL1_MCU_AMUX1_3P3: now also U11.12 (PF2); no longer U11.73 (PB12)
- net GPIO_SEL1_MCU_AMUX3_3P3: now also U11.89 (PG4); no longer U11.109 (PA14)
- net GPIO_SEL_MCU_AMUX2_3P3: now also U11.65 (PE12); no longer U11.119 (PD5)
- net GPIO_SW-SEL_MCU_CLKMUX_3P3: now also U11.67 (PE14); no longer U11.123 (PD7)
- net GPIO_W-CLK_MCU_DDS_3P3: now also U11.79 (PD10); no longer U11.71 (VCAP_1)
- net I2C_SCL_MCU_POT_3P3: now also U11.69 (PB10); no longer U11.10 (PF0)
- net I2C_SDA_MCU_POT_3P3: now also U11.70 (PB11); no longer U11.11 (PF1)
- net JTAG_MCU_TCK_3P3: now also U11.109 (PA14); no longer U11.89 (PG4)
- net JTAG_MCU_TDI_3P3: now also U11.110 (PA15); no longer U11.90 (PG5)
- net JTAG_MCU_TDO_3P3: now also U11.133 (PB3); no longer U11.125 (PG10)
- net JTAG_MCU_TMS_3P3: now also U11.105 (PA13); no longer U11.88 (PG3)
- net QSPI_IO0_MCU_FLASH_3P3: now also U11.20 (PF8); no longer U11.27 (PC1)
- net QSPI_IO1_MCU_FLASH_3P3: now also U11.21 (PF9); no longer U11.28 (PC2)
- net QSPI_IO2_MCU_FLASH_3P3: now also U11.1 (PE2); no longer U11.113 (PC12)
- net QSPI_IO3_MCU_FLASH_3P3: now also U11.18 (PF6)
- net QSPI_NCS_MCU_FLASH_3P3: now also U11.91 (PG6)
- net SPI_CS_MCU_FLASH_3P3_L: now also U11.29 (PC3)
- net SPI_CS_MCU_FPGA_3P3_L: now also U11.26 (PC0)
- net SPI_MISO_FPGA_MCU_3P3: now also U11.28 (PC2); no longer U11.21 (PF9)
- net SPI_MOSI_MCU_FPGA_3P3: now also U11.27 (PC1); no longer U11.20 (PF8)
- net SPI_SCLK_MCU_FPGA_3P3: now also U11.74 (PB13); no longer U11.13 (PF3)
- net UART_FTDITX_MCURX_3P3: now also U11.37 (PA3); no longer U11.138 (BOOT0)
- net UART_MCUTX_FTDIRX_3P3: now also U11.36 (PA2)
- net at C38.1: now also U11.71 (VCAP_1); no longer U11.79 (PD10)
- net at C43.1, Y1.1: now also U11.9 (PC15); no longer U11.4 (PE5)
- net at C45.1, Y1.2: now also U11.8 (PC14); no longer U11.3 (PE4)
- net at R31.2: now also U11.143 (PDR_ON); no longer U11.35 (PA1)
- net at U11.106 (VCAP_2): now also C39.1
- net at U11.80 (PD11): no longer C39.1
Changed lines of the file:
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@@
 		)
 	)
-	(global_label "SPI_SCLK_MCU_FPGA_3P3"
+	(global_label "GPIO_SW-SEL_MCU_CLKMUX_3P3"
 		(shape input)
-		(at 111.76 105.41 0)
+		(at 50.8 176.53 180)
 		(fields_autoplaced yes)
 		(effects
@@
 				(size 1.27 1.27)
 			)
-			(justify left)
+			(justify right)
 		)
 		(property "Intersheetrefs" "${INTERSHEET_REFS}"
-			(at 138.9356 105.41 0)
+			(at 16.5488 176.53 0)
 			(effects
 				(font
 					(size 1.27 1.27)
 				)
-				(justify left)
+				(justify right)
 				(hide yes)
 			)
 		)
 	)
-	(global_label "GPIO_SW-SEL_MCU_CLKMUX_3P3"
+	(global_label "GPIO_CLK_EN_MCU_FPGA_3P3"
 		(shape input)
-		(at 50.8 176.53 180)
+		(at 50.8 163.83 180)
 		(fields_autoplaced yes)
 		(effects
@@
 		)
 		(property "Intersheetrefs" "${INTERSHEET_REFS}"
-			(at 16.5488 176.53 0)
+			(at 19.9958 163.83 0)
 			(effects
 				(font
@@
 		)
 	)
-	(global_label "GPIO_CLK_EN_MCU_FPGA_3P3"
+	(global_label "JTAG_MCU_TCK_3P3"
 		(shape input)
-		(at 50.8 163.83 180)
+		(at 111.76 64.77 0)
+		(fields_autoplaced yes)
+		(effects
+			(font
+				(size 1.27 1.27)
+			)
+			(justify left)
+		)
+		(property "Intersheetrefs" "${INTERSHEET_REFS}"
+			(at 133.1903 64.77 0)
+			(effects
+				(font
+					(size 1.27 1.27)
+				)
+				(justify left)
+				(hide yes)
+			)
+		)
+	)
+	(global_label "GPIO_100M-EN_MCU_100M-OSC_3P3"
+		(shape input)
+		(at 50.8 173.99 180)
 		(fields_autoplaced yes)
 		(effects
@@
 		)
 		(property "Intersheetrefs" "${INTERSHEET_REFS}"
-			(at 19.9958 163.83 0)
+			(at 12.1341 173.99 0)
 			(effects
 				(font
@@
 		)
 	)
-	(global_label "JTAG_MCU_TCK_3P3"
+	(global_label "SPI_CS_MCU_FLASH_3P3_L"
 		(shape input)
-		(at 111.76 64.77 0)
+		(at 111.76 123.19 0)
 		(fields_autoplaced yes)
 		(effects
@@
 		)
 		(property "Intersheetrefs" "${INTERSHEET_REFS}"
-			(at 133.1903 64.77 0)
+			(at 139.6613 123.19 0)
 			(effects
 				(font
@@
 		)
 	)
-	(global_label "GPIO_100M-EN_MCU_100M-OSC_3P3"
+	(global_label "SPI_SCLK_MCU_FPGA_3P3"
 		(shape input)
-		(at 50.8 173.99 180)
+		(at 111.76 105.41 0)
 		(fields_autoplaced yes)
 		(effects
@@
 				(size 1.27 1.27)
 			)
-			(justify right)
+			(justify left)
 		)
 		(property "Intersheetrefs" "${INTERSHEET_REFS}"
-			(at 12.1341 173.99 0)
+			(at 138.9356 105.41 0)
 			(effects
 				(font
 					(size 1.27 1.27)
 				)
-				(justify right)
+				(justify left)
 				(hide yes)
 			)
@@
 		)
 	)
-	(global_label "SPI_CS_MCU_FPGA_3P3_L"
-		(shape input)
-		(at 149.86 118.11 0)
-		(fields_autoplaced yes)
-		(effects
-			(font
-				(size 1.27 1.27)
-			)
-			(justify left)
-		)
-		(property "Intersheetrefs" "${INTERSHEET_REFS}"
-			(at 176.7332 118.11 0)
-			(effects
-				(font
-					(size 1.27 1.27)
-				)
-				(justify left)
-				(hide yes)
-			)
-		)
-	)
 	(global_label "GPIO_D7_MCU_DDS_3P3"
 		(shape input)
@@
 		)
 	)
-	(global_label "SPI_CS_MCU_FLASH_3P3_L"
+	(global_label "SPI_CS_MCU_FPGA_3P3_L"
 		(shape input)
-		(at 149.86 125.73 0)
+		(at 111.76 115.57 0)
 		(fields_autoplaced yes)
 		(effects
@@
 		)
 		(property "Intersheetrefs" "${INTERSHEET_REFS}"
-			(at 177.7613 125.73 0)
+			(at 138.6332 115.57 0)
 			(effects
 				(font
@@
 		(lib_id "BRZK_STM32:STM32F446ZETx")
 		(at 81.28 115.57 0)
-		(mirror y)
 		(unit 1)
 		(exclude_from_sim no)
@@
 		(dnp no)
 		(property "Reference" "U11"
-			(at 109.22 20.32 0)
+			(at 53.34 20.32 0)
 			(effects
 				(font
@@
 		)
 		(property "Value" "STM32F446ZETx"
-			(at 109.22 22.86 0)
+			(at 53.34 22.86 0)
 			(effects
 				(font
@@
 		)
 		(property "Footprint" "Package_QFP:LQFP-144_20x20mm_P0.5mm"
-			(at 106.68 201.93 0)
+			(at 55.88 201.93 0)
 			(effects
 				(font

Commit message: FEAT: Finished DDS, MCU Layout.
Connections:
- net GPIO_100M-EN_MCU_100M-OSC_3P3: now also U11.73 (PB12); no longer U11.66 (PE13)
- net GPIO_AMP-PD_MCU_AMP2_3P3: now also U11.58 (PE7); no longer U11.56 (PG0)
- net GPIO_CFG_DONE_FPGA_MCU_3P3: now also U11.56 (PG0); no longer U11.58 (PE7)
- net GPIO_CLK_EN_MCU_FPGA_3P3: now also U11.59 (PE8); no longer U11.60 (PE9)
- net GPIO_D0_MCU_DDS_3P3: now also U11.88 (PG3); no longer U11.114 (PD0)
- net GPIO_D1_MCU_DDS_3P3: now also U11.89 (PG4); no longer U11.115 (PD1)
- net GPIO_D2_MCU_DDS_3P3: now also U11.90 (PG5); no longer U11.116 (PD2)
- net GPIO_D3_MCU_DDS_3P3: now also U11.103 (PA11); no longer U11.117 (PD3)
- net GPIO_D4_MCU_DDS_3P3: now also U11.79 (PD10); no longer U11.118 (PD4)
- net GPIO_D5_MCU_DDS_3P3: now also U11.78 (PD9); no longer U11.119 (PD5)
- net GPIO_D6_MCU_DDS_3P3: now also U11.77 (PD8); no longer U11.122 (PD6)
- net GPIO_D7_MCU_DDS_3P3: now also U11.76 (PB15); no longer U11.123 (PD7)
- net GPIO_EN_MCU_AMUX1_3P3: now also U11.46 (PB0); no longer U11.10 (PF0)
- net GPIO_EN_MCU_AMUX2_3P3: now also U11.66 (PE13); no longer U11.64 (PE11)
- net GPIO_EN_MCU_AMUX3_3P3: now also U11.35 (PA1); no longer U11.88 (PG3)
- net GPIO_FPGARST_MCU_FPGA_3P3_L: now also U11.57 (PG1); no longer U11.59 (PE8)
- net GPIO_FQ-UD_MCU_DDS_3P3: now also U11.87 (PG2); no longer U11.78 (PD9)
- net GPIO_RST_MCU_DDS_3P3: now also U11.75 (PB14); no longer U11.77 (PD8)
- net GPIO_SEL0_MCU_AMUX1_3P3: now also U11.44 (PC4); no longer U11.11 (PF1)
- net GPIO_SEL0_MCU_AMUX3_3P3: now also U11.34 (PA0); no longer U11.90 (PG5)
- net GPIO_SEL1_MCU_AMUX1_3P3: now also U11.45 (PC5); no longer U11.12 (PF2)
- net GPIO_SEL1_MCU_AMUX3_3P3: now also U11.43 (PA7); no longer U11.89 (PG4)
- net GPIO_SEL_MCU_AMUX2_3P3: now also U11.67 (PE14); no longer U11.65 (PE12)
- net GPIO_SW-SEL_MCU_CLKMUX_3P3: now also U11.112 (PC11); no longer U11.67 (PE14)
- net GPIO_W-CLK_MCU_DDS_3P3: now also U11.104 (PA12); no longer U11.79 (PD10)
- no-connect marks 65 -> 49
