File: 1_hw/03_pcb/connectors.kicad_sch (KiCad schematic)
At the start: 19 parts, among them J1 TYPE-C-31-M-12, J2 SMA, J3 SMA, J4 BNC, J5 PH-00244

Commit message: FEAT: Initial board placement started.
Parts:
- H1, H2, H3, H4: footprint MountingHole_3.2mm_M3_Pad -> MountingHole:MountingHole_3.2mm_M3_Pad
Changed lines of the file:
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@@
 		(dnp no)
 		(fields_autoplaced yes)
-		(property "Reference" "#PWR0284"
+		(property "Reference" "#PWR0296"
 			(at 35.56 121.92 0)
 			(effects
@@
 			(project "arb"
 				(path "/866ef9be-3b01-4288-a6e0-a2357aa17e50/eb105004-087f-4ea7-8291-809b214299af"
-					(reference "#PWR0284")
+					(reference "#PWR0296")
 					(unit 1)
 				)
@@
 			)
 		)
-		(property "Footprint" "MountingHole_3.2mm_M3_Pad"
+		(property "Footprint" "MountingHole:MountingHole_3.2mm_M3_Pad"
 			(at 242.57 17.78 0)
 			(effects
@@
 		(dnp no)
 		(fields_autoplaced yes)
-		(property "Reference" "#PWR0286"
+		(property "Reference" "#PWR0298"
 			(at 36.83 163.83 0)
 			(effects
@@
 			(project "arb"
 				(path "/866ef9be-3b01-4288-a6e0-a2357aa17e50/eb105004-087f-4ea7-8291-809b214299af"
-					(reference "#PWR0286")
+					(reference "#PWR0298")
 					(unit 1)
 				)
@@
 		(dnp no)
 		(fields_autoplaced yes)
-		(property "Reference" "#PWR0294"
+		(property "Reference" "#PWR0306"
 			(at 260.35 25.4 0)
 			(effects
@@
 			(project "arb"
 				(path "/866ef9be-3b01-4288-a6e0-a2357aa17e50/eb105004-087f-4ea7-8291-809b214299af"
-					(reference "#PWR0294")
+					(reference "#PWR0306")
 					(unit 1)
 				)
@@
 		(dnp no)
 		(fields_autoplaced yes)
-		(property "Reference" "#PWR0289"
+		(property "Reference" "#PWR0301"
 			(at 82.55 45.72 0)
 			(effects
@@
 			(project "arb"
 				(path "/866ef9be-3b01-4288-a6e0-a2357aa17e50/eb105004-087f-4ea7-8291-809b214299af"
-					(reference "#PWR0289")
+					(reference "#PWR0301")
 					(unit 1)
 				)
@@
 		(dnp no)
 		(fields_autoplaced yes)
-		(property "Reference" "#PWR0285"
+		(property "Reference" "#PWR0297"
 			(at 35.56 146.05 0)
 			(effects
@@
 			(project "arb"
 				(path "/866ef9be-3b01-4288-a6e0-a2357aa17e50/eb105004-087f-4ea7-8291-809b214299af"
-					(reference "#PWR0285")
+					(reference "#PWR0297")
 					(unit 1)
 				)
@@
 			)
 		)
-		(property "Footprint" "MountingHole_3.2mm_M3_Pad"
+		(property "Footprint" "MountingHole:MountingHole_3.2mm_M3_Pad"
 			(at 232.41 17.78 0)
 			(effects
@@
 		(dnp no)
 		(fields_autoplaced yes)
-		(property "Reference" "#PWR0291"
+		(property "Reference" "#PWR0303"
 			(at 232.41 25.4 0)
 			(effects
@@
 			(project "arb"
 				(path "/866ef9be-3b01-4288-a6e0-a2357aa17e50/eb105004-087f-4ea7-8291-809b214299af"
-					(reference "#PWR0291")
+					(reference "#PWR0303")
 					(unit 1)
 				)
@@
 		(dnp no)
 		(fields_autoplaced yes)
-		(property "Reference" "#PWR0293"
+		(property "Reference" "#PWR0305"
 			(at 251.46 25.4 0)
 			(effects
@@
 			(project "arb"
 				(path "/866ef9be-3b01-4288-a6e0-a2357aa17e50/eb105004-087f-4ea7-8291-809b214299af"
-					(reference "#PWR0293")
+					(reference "#PWR0305")
 					(unit 1)
 				)
@@
 			)
 		)
-		(property "Footprint" "MountingHole_3.2mm_M3_Pad"
+		(property "Footprint" "MountingHole:MountingHole_3.2mm_M3_Pad"
 			(at 251.46 17.78 0)
 			(effects
@@
 		(dnp no)
 		(fields_autoplaced yes)
-		(property "Reference" "#PWR0287"
+		(property "Reference" "#PWR0299"
 			(at 36.83 179.07 0)
 			(effects
@@
 			(project "arb"
 				(path "/866ef9be-3b01-4288-a6e0-a2357aa17e50/eb105004-087f-4ea7-8291-809b214299af"
-					(reference "#PWR0287")
+					(reference "#PWR0299")
 					(unit 1)
 				)
@@
 		(dnp no)
 		(fields_autoplaced yes)
-		(property "Reference" "#PWR0292"
+		(property "Reference" "#PWR0304"
 			(at 242.57 25.4 0)
 			(effects
@@
 			(project "arb"
 				(path "/866ef9be-3b01-4288-a6e0-a2357aa17e50/eb105004-087f-4ea7-8291-809b214299af"
-					(reference "#PWR0292")
+					(reference "#PWR0304")
 					(unit 1)
 				)
@@
 		(dnp no)
 		(fields_autoplaced yes)
-		(property "Reference" "#PWR0290"
+		(property "Reference" "#PWR0302"
 			(at 91.44 45.72 0)
 			(effects
@@
 			(project "arb"
 				(path "/866ef9be-3b01-4288-a6e0-a2357aa17e50/eb105004-087f-4ea7-8291-809b214299af"
-					(reference "#PWR0290")
+					(reference "#PWR0302")
 					(unit 1)
 				)
@@
 		(dnp no)
 		(fields_autoplaced yes)
-		(property "Reference" "#PWR0281"
+		(property "Reference" "#PWR0293"
 			(at 25.4 69.85 0)
 			(effects
@@
 			(project "arb"
 				(path "/866ef9be-3b01-4288-a6e0-a2357aa17e50/eb105004-087f-4ea7-8291-809b214299af"
-					(reference "#PWR0281")
+					(reference "#PWR0293")
 					(unit 1)
 				)
@@
 		(dnp no)
 		(fields_autoplaced yes)
-		(property "Reference" "#PWR0282"
+		(property "Reference" "#PWR0294"
 			(at 33.02 71.12 0)
 			(effects
@@
 			(project "arb"
 				(path "/866ef9be-3b01-4288-a6e0-a2357aa17e50/eb105004-087f-4ea7-8291-809b214299af"
-					(reference "#PWR0282")
+					(reference "#PWR0294")
 					(unit 1)
 				)
@@
 			)
 		)
-		(property "Footprint" "MountingHole_3.2mm_M3_Pad"
+		(property "Footprint" "MountingHole:MountingHole_3.2mm_M3_Pad"
 			(at 260.35 17.78 0)
 			(effects
@@
 		(dnp no)
 		(fields_autoplaced yes)
-		(property "Reference" "#PWR0288"
+		(property "Reference" "#PWR0300"
 			(at 55.88 29.21 0)
 			(effects
@@
 			(project "arb"
 				(path "/866ef9be-3b01-4288-a6e0-a2357aa17e50/eb105004-087f-4ea7-8291-809b214299af"
-					(reference "#PWR0288")
+					(reference "#PWR0300")
 					(unit 1)
 				)
@@
 		(dnp no)
 		(fields_autoplaced yes)
-		(property "Reference" "#PWR0283"
+		(property "Reference" "#PWR0295"
 			(at 35.56 97.79 0)
 			(effects
@@
 			(project "arb"
 				(path "/866ef9be-3b01-4288-a6e0-a2357aa17e50/eb105004-087f-4ea7-8291-809b214299af"
-					(reference "#PWR0283")
-					(unit 1)
-				)
+					(reference "#PWR0295")
+					(unit 1)
+				)

Commit message: FEAT: Removed Chassis GND, completed routing. Needs to be verified.
Connections:
- net C_GND is gone; now on net GND: H1.1, H2.1, H3.1, H4.1, J1.S1 (SHIELD), J2.2 (Ext), J3.2 (Ext), J4.2 (Ext)
