File: 2_HARDWARE/03_PCB/analog2.kicad_sch (KiCad schematic)
At the start: 19 parts, among them U22 TPL0401B-10, U23 THS3491, U24 ADG1219BRJZ

Commit message: MINOR: Adjusted Analog Schematic.
Parts:
- added R6, R98: 0, Resistor_SMD:R_0603_1608Metric, symbol Device:R_Small_US
Connections:
- net ANALOG_DC-OFFSET_AMUX3_AMP3: now also R6.1; no longer U22.6 (H), U23.2 (-)
- new net: R98.2, U22.6 (H), U23.2 (-)
- new net: R6.2, R98.1
Other:
- note added: "R6: PLACEHOLDER TUNING CAP FOR DC BLOCKING R98: PLACEHOLDER TUNING RESISTOR FOR ADJUSTING FEEDBACK GAIN"
Changed lines of the file:
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@@
+		)
+	)
+	(text "R6: PLACEHOLDER TUNING CAP FOR DC BLOCKING\nR98: PLACEHOLDER TUNING RESISTOR FOR ADJUSTING FEEDBACK GAIN"
+		(exclude_from_sim no)
+		(at 20.32 72.39 0)
+		(effects
+			(font
+				(size 1.27 1.27)
+			)
+			(justify left)
 		)
 	)
@@
 	(wire
 		(pts
-			(xy 54.61 60.96) (xy 64.77 60.96)
+			(xy 54.61 78.74) (xy 64.77 78.74)
 		)
 		(stroke
@@
 	(wire
 		(pts
+			(xy 79.0666 86.36) (xy 73.66 86.36)
+		)
+		(stroke
+			(width 0)
+			(type default)
+		)
+	)
+	(wire
+		(pts
 			(xy 62.23 118.11) (xy 62.23 129.54)
 		)
@@
 	(wire
 		(pts
-			(xy 97.79 86.36) (xy 64.77 86.36)
+			(xy 97.79 86.36) (xy 84.1466 86.36)
 		)
 		(stroke
@@
 	(wire
 		(pts
+			(xy 68.58 86.36) (xy 64.77 86.36)
+		)
+		(stroke
+			(width 0)
+			(type default)
+		)
+	)
+	(wire
+		(pts
 			(xy 170.18 139.7) (xy 173.99 139.7)
 		)
@@
 	(wire
 		(pts
-			(xy 64.77 60.96) (xy 64.77 86.36)
+			(xy 64.77 78.74) (xy 64.77 86.36)
 		)
 		(stroke
@@
 	(global_label "ANALOG_DC-OFFSET_AMUX3_AMP3"
 		(shape input)
-		(at 54.61 60.96 180)
+		(at 54.61 78.74 180)
 		(fields_autoplaced yes)
 		(effects
@@
 		)
 		(property "Intersheetrefs" "${INTERSHEET_REFS}"
-			(at 19.3305 60.96 0)
+			(at 19.3305 78.74 0)
 			(effects
 				(font
@@
 	)
 	(symbol
+		(lib_id "Device:R_Small_US")
+		(at 71.12 86.36 90)
+		(unit 1)
+		(exclude_from_sim no)
+		(in_bom yes)
+		(on_board yes)
+		(dnp no)
+		(fields_autoplaced yes)
+		(property "Reference" "R6"
+			(at 71.12 80.01 90)
+			(effects
+				(font
+					(size 1.27 1.27)
+				)
+			)
+		)
+		(property "Value" "0"
+			(at 71.12 82.55 90)
+			(effects
+				(font
+					(size 1.27 1.27)
+				)
+			)
+		)
+		(property "Footprint" "Resistor_SMD:R_0603_1608Metric"
+			(at 71.12 86.36 0)
+			(effects
+				(font
+					(size 1.27 1.27)
+				)
+				(hide yes)
+			)
+		)
+		(property "Datasheet" "~"
+			(at 71.12 86.36 0)
+			(effects
+				(font
+					(size 1.27 1.27)
+				)
+				(hide yes)
+			)
+		)
+		(property "Description" "Resistor, small US symbol"
+			(at 71.12 86.36 0)
+			(effects
+				(font
+					(size 1.27 1.27)
+				)
+				(hide yes)
+			)
+		)
+		(property "Part Number" "0603WAJ0000T5E"
+			(at 71.12 86.36 0)
+			(effects
+				(font
+					(size 1.27 1.27)
+				)
+				(hide yes)
+			)
+		)
+		(property "LCSC" "C15402"
+			(at 71.12 86.36 0)
+			(effects
+				(font
+					(size 1.27 1.27)
+				)
+				(hide yes)
+			)
+		)
+		(pin "2"
+		)
+		(pin "1"
+		)
+		(instances
+			(project "arb"
+				(path "/866ef9be-3b01-4288-a6e0-a2357aa17e50/e46c6640-71a3-4b78-b602-0f6be9676e36"
+					(reference "R6")
+					(unit 1)
+				)
+			)
+		)
+	)
+	(symbol
 		(lib_id "Device:C_Small")
 		(at 152.4 95.25 0)
@@
 					(unit 1)
 				)
+			)
+		)
+	)
+	(symbol
+		(lib_id "Device:R_Small_US")
+		(at 81.6066 86.36 90)
+		(unit 1)
+		(exclude_from_sim no)
+		(in_bom yes)
+		(on_board yes)
+		(dnp no)
+		(fields_autoplaced yes)
+		(property "Reference" "R98"
+			(at 81.6066 80.01 90)
+			(effects
+				(font
+					(size 1.27 1.27)
+				)
+			)
+		)
+		(property "Value" "0"
+			(at 81.6066 82.55 90)
+			(effects
+				(font
+					(size 1.27 1.27)
+				)
+			)
+		)
+		(property "Footprint" "Resistor_SMD:R_0603_1608Metric"
+			(at 81.6066 86.36 0)
+			(effects
+				(font
+					(size 1.27 1.27)
+				)
+				(hide yes)
+			)
+		)
+		(property "Datasheet" "~"
+			(at 81.6066 86.36 0)
+			(effects
+				(font
+					(size 1.27 1.27)
+				)
+				(hide yes)
+			)
+		)
+		(property "Description" "Resistor, small US symbol"
+			(at 81.6066 86.36 0)
+			(effects
+				(font
+					(size 1.27 1.27)
+				)
+				(hide yes)
+			)
+		)
+		(property "Part Number" "0603WAJ0000T5E"
+			(at 81.6066 86.36 0)
+			(effects
+				(font
+					(size 1.27 1.27)
+				)
+				(hide yes)
+			)
+		)
+		(property "LCSC" "C15402"
+			(at 81.6066 86.36 0)
+			(effects
+				(font
+					(size 1.27 1.27)
+				)
+				(hide yes)
+			)
+		)
+		(pin "2"
+		)
+		(pin "1"
+		)
+		(instances
+			(project "arb"
+				(path "/866ef9be-3b01-4288-a6e0-a2357aa17e50/e46c6640-71a3-4b78-b602-0f6be9676e36"
+					(reference "R98")
+					(unit 1)
+				)
