File: 2_HARDWARE/03_PCB/analog1.kicad_sch (KiCad schematic)
At the start: 26 parts, among them U19 LM6171, U20 LM6171, U21 TMUX6104

Commit message: MINOR: Changed Boot Select Switches to Pull-Downs / Pull Up DNI and continued layout.
Parts:
- renumbered R60 to R61, R61 to R62, R62 to R63, R63 to R64, R64 to R65, R65 to R66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
