File: 2_HARDWARE/03_PCB/arb.kicad_pcb (KiCad board)
At the start: 4 copper layers, 104.3 x 53.5 mm, 269 parts, among them J1 TYPE-C-31-M-12, J2 SMA, J3 SMA, J4 BNC, J5 PH-00244, SW1 TS-1187A-B-A-B, U1 TLV70333DBV, U10 LMK1C1103PWR, U11 STM32F446ZETx, U12 ICE40UP5K-SG48ITR, U13 93LC56BT-I_OT, U14 FT2232HL, U15 W25Q128JVSIQ, U16 W25Q128JVSIQ, U17 AD9850, U18 AD9744, U19 LM6171, U2 TLV76133DCY, U20 LM6171, U21 TMUX6104, U22 TPL0401B-10, U23 THS3491, U24 ADG1219BRJZ, U25 LM6171, U26 TMUX6104, U3 TLV70333DBV, U4 LM3880MF-1AA, U5 TLV70312DBV, U6 TLV70325DBV, U7 TPS65131RGE, U8 TPD2E001DRL, U9 ADG1219BRJZ, X1 ASE-10.000MHz, X2 ASE-100.000MHz, Y1 32.768k, Y2 12 MHz

Commit message: MINOR: Completed initial placement.
Parts:
- moved R87 96.5 mm to (160.5, 79.0), turned to -90 degrees
- moved R86 95.7 mm to (162.8, 79.8), turned to 180 degrees
- moved C111 94.2 mm to (149.5, 79.5), turned to 180 degrees
- moved U25 92.1 mm to (155.0, 80.5), turned to 180 degrees
- moved R89 91.2 mm to (149.5, 81.0), turned to 180 degrees
- moved C112 84.1 mm to (158.5, 84.9), turned to -90 degrees
- moved R88 80.9 mm to (154.8, 86.2), turned to 180 degrees
- moved C113 80.1 mm to (153.0, 90.8), turned to 90 degrees
- moved R85 77.9 mm to (154.8, 87.7), turned to 180 degrees
- moved D8 77.1 mm to (135.0, 86.2)
- moved D7 75.6 mm to (131.0, 86.2)
- moved R53 75.6 mm to (133.0, 85.7), turned to 90 degrees
- moved R52 74.2 mm to (129.1, 85.7), turned to 90 degrees
- moved U26 73.0 mm to (152.5, 96.5), turned to 90 degrees
- moved R90 71.9 mm to (157.3, 101.7), turned to 180 degrees
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