File: 2_HARDWARE/03_PCB/power.kicad_sch (KiCad schematic)
At the start: 62 parts, among them U1 TLV70333DBV, U2 TLV76133DCY, U3 TLV70333DBV, U4 LM3880MF-1AA, U5 TLV70312DBV, U6 TLV70325DBV, U7 TPS65131RGE, U8 TPD2E001DRL

Commit message: MINOR: Changed Boot Select Switches to Pull-Downs / Pull Up DNI and continued layout.
Parts:
- renumbered R11 to R10, R12 to R11, R13 to R12, R14 to R13, R15 to R14, R16 to R15, R17 to R16, R18 to R17, R7 to R6, R8 to R7, R9 to R8, R10 to R9

Commit message: MINORL: Completed 3.3V Regulator Power Planes. Started on FTDI Clock.
Changed lines of the file:
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@@
 		(lib_id "power:+3V3")
 		(at 259.08 83.82 0)
+		(mirror y)
 		(unit 1)
 		(exclude_from_sim no)
@@
 		(on_board yes)
 		(dnp no)
-		(fields_autoplaced yes)
 		(property "Reference" "#PWR068"
 			(at 259.08 87.63 0)
