File: 2_HARDWARE/03_PCB/ftdi.kicad_sch (KiCad schematic)
At the start: 34 parts, among them U13 93LC56BT-I_OT, U14 FT2232HL, Y2 12 MHz

Commit message: MINOR: Changed Boot Select Switches to Pull-Downs / Pull Up DNI and continued layout.
Parts:
- renumbered R41 to R42, R42 to R43, R43 to R44, R44 to R45, R45 to R46, R46 to R47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
