File: 2_HARDWARE/03_PCB/analogdc.kicad_sch (KiCad schematic)
At the start: 12 parts, among them U25 LM6171, U26 TMUX6104

Commit message: MINOR: Changed Boot Select Switches to Pull-Downs / Pull Up DNI and continued layout.
Parts:
- renumbered R82 to R85, R83 to R86, R84 to R87, R85 to R88, R86 to R89, R87 to R90
Changed lines of the file:
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@@
 		(dnp no)
 		(fields_autoplaced yes)
-		(property "Reference" "R87"
+		(property "Reference" "R90"
 			(at 186.69 110.4899 0)
 			(effects
@@
 			(project "arb"
 				(path "/866ef9be-3b01-4288-a6e0-a2357aa17e50/dd20ed2c-105a-40ef-bdba-a4198899f68e"
-					(reference "R87")
+					(reference "R90")
 					(unit 1)
 				)
@@
 		(on_board yes)
 		(dnp no)
-		(property "Reference" "#PWR0291"
+		(property "Reference" "#PWR0287"
 			(at 209.55 121.92 0)
 			(effects
@@
 			(project "arb"
 				(path "/866ef9be-3b01-4288-a6e0-a2357aa17e50/dd20ed2c-105a-40ef-bdba-a4198899f68e"
-					(reference "#PWR0291")
+					(reference "#PWR0287")
 					(unit 1)
 				)
@@
 		(on_board yes)
 		(dnp no)
-		(property "Reference" "#PWR0289"
+		(property "Reference" "#PWR0285"
 			(at 191.77 121.92 0)
 			(effects
@@
 			(project "arb"
 				(path "/866ef9be-3b01-4288-a6e0-a2357aa17e50/dd20ed2c-105a-40ef-bdba-a4198899f68e"
-					(reference "#PWR0289")
+					(reference "#PWR0285")
 					(unit 1)
 				)
@@
 		(dnp no)
 		(fields_autoplaced yes)
-		(property "Reference" "R84"
+		(property "Reference" "R87"
 			(at 92.71 107.9499 0)
 			(effects
@@
 			(project "arb"
 				(path "/866ef9be-3b01-4288-a6e0-a2357aa17e50/dd20ed2c-105a-40ef-bdba-a4198899f68e"
-					(reference "R84")
+					(reference "R87")
 					(unit 1)
 				)
@@
 		(dnp no)
 		(fields_autoplaced yes)
-		(property "Reference" "#PWR0282"
+		(property "Reference" "#PWR0278"
 			(at 40.64 107.95 0)
 			(effects
@@
 			(project "arb"
 				(path "/866ef9be-3b01-4288-a6e0-a2357aa17e50/dd20ed2c-105a-40ef-bdba-a4198899f68e"
-					(reference "#PWR0282")
+					(reference "#PWR0278")
 					(unit 1)
 				)
@@
 		(dnp no)
 		(fields_autoplaced yes)
-		(property "Reference" "#PWR0293"
+		(property "Reference" "#PWR0289"
 			(at 213.36 87.63 0)
 			(effects
@@
 			(project "arb"
 				(path "/866ef9be-3b01-4288-a6e0-a2357aa17e50/dd20ed2c-105a-40ef-bdba-a4198899f68e"
-					(reference "#PWR0293")
+					(reference "#PWR0289")
 					(unit 1)
 				)
@@
 		(on_board yes)
 		(dnp no)
-		(property "Reference" "R83"
+		(property "Reference" "R86"
 			(at 78.74 108.204 90)
 			(effects
@@
 			(project "arb"
 				(path "/866ef9be-3b01-4288-a6e0-a2357aa17e50/dd20ed2c-105a-40ef-bdba-a4198899f68e"
-					(reference "R83")
+					(reference "R86")
 					(unit 1)
 				)
@@
 		(dnp no)
 		(fields_autoplaced yes)
-		(property "Reference" "R85"
+		(property "Reference" "R88"
 			(at 106.68 69.85 90)
 			(effects
@@
 			(project "arb"
 				(path "/866ef9be-3b01-4288-a6e0-a2357aa17e50/dd20ed2c-105a-40ef-bdba-a4198899f68e"
-					(reference "R85")
+					(reference "R88")
 					(unit 1)
 				)
@@
 		(dnp no)
 		(fields_autoplaced yes)
-		(property "Reference" "#PWR0283"
+		(property "Reference" "#PWR0279"
 			(at 90.17 118.11 0)
 			(effects
@@
 			(project "arb"
 				(path "/866ef9be-3b01-4288-a6e0-a2357aa17e50/dd20ed2c-105a-40ef-bdba-a4198899f68e"
-					(reference "#PWR0283")
+					(reference "#PWR0279")
 					(unit 1)
 				)
@@
 		(dnp no)
 		(fields_autoplaced yes)
-		(property "Reference" "#PWR0287"
+		(property "Reference" "#PWR0283"
 			(at 109.22 123.19 0)
 			(effects
@@
 			(project "arb"
 				(path "/866ef9be-3b01-4288-a6e0-a2357aa17e50/dd20ed2c-105a-40ef-bdba-a4198899f68e"
-					(reference "#PWR0287")
+					(reference "#PWR0283")
 					(unit 1)
 				)
@@
 		(dnp no)
 		(fields_autoplaced yes)
-		(property "Reference" "#PWR0285"
+		(property "Reference" "#PWR0281"
 			(at 104.14 116.84 0)
 			(effects
@@
 			(project "arb"
 				(path "/866ef9be-3b01-4288-a6e0-a2357aa17e50/dd20ed2c-105a-40ef-bdba-a4198899f68e"
-					(reference "#PWR0285")
+					(reference "#PWR0281")
 					(unit 1)
 				)
@@
 		(dnp no)
 		(fields_autoplaced yes)
-		(property "Reference" "#PWR0284"
+		(property "Reference" "#PWR0280"
 			(at 104.14 88.9 0)
 			(effects
@@
 			(project "arb"
 				(path "/866ef9be-3b01-4288-a6e0-a2357aa17e50/dd20ed2c-105a-40ef-bdba-a4198899f68e"
-					(reference "#PWR0284")
+					(reference "#PWR0280")
 					(unit 1)
 				)
@@
 		(dnp no)
 		(fields_autoplaced yes)
-		(property "Reference" "#PWR0288"
+		(property "Reference" "#PWR0284"
 			(at 184.15 120.65 0)
 			(effects
@@
 			(project "arb"
 				(path "/866ef9be-3b01-4288-a6e0-a2357aa17e50/dd20ed2c-105a-40ef-bdba-a4198899f68e"
-					(reference "#PWR0288")
+					(reference "#PWR0284")
 					(unit 1)
 				)
@@
 		(on_board yes)
 		(dnp no)
-		(property "Reference" "R82"
+		(property "Reference" "R85"
 			(at 78.74 93.98 90)
 			(effects
@@
 			(project "arb"
 				(path "/866ef9be-3b01-4288-a6e0-a2357aa17e50/dd20ed2c-105a-40ef-bdba-a4198899f68e"
-					(reference "R82")
+					(reference "R85")
 					(unit 1)
 				)
@@
 		(dnp no)
 		(fields_autoplaced yes)
-		(property "Reference" "R86"
+		(property "Reference" "R89"
 			(at 127 96.52 90)
 			(effects
@@
 			(project "arb"
 				(path "/866ef9be-3b01-4288-a6e0-a2357aa17e50/dd20ed2c-105a-40ef-bdba-a4198899f68e"
-					(reference "R86")
+					(reference "R89")
 					(unit 1)
 				)
@@
 		(dnp no)
 		(fields_autoplaced yes)
-		(property "Reference" "#PWR0290"
+		(property "Reference" "#PWR0286"
 			(at 209.55 78.74 0)
 			(effects
@@
 			(project "arb"
 				(path "/866ef9be-3b01-4288-a6e0-a2357aa17e50/dd20ed2c-105a-40ef-bdba-a4198899f68e"
-					(reference "#PWR0290")
+					(reference "#PWR0286")
 					(unit 1)
 				)
@@
 		(dnp no)
 		(fields_autoplaced yes)
-		(property "Reference" "#PWR0292"
+		(property "Reference" "#PWR0288"
 			(at 212.09 121.92 0)
 			(effects
@@
 			(project "arb"
 				(path "/866ef9be-3b01-4288-a6e0-a2357aa17e50/dd20ed2c-105a-40ef-bdba-a4198899f68e"
-					(reference "#PWR0292")
+					(reference "#PWR0288")
 					(unit 1)
 				)
@@
 		(dnp no)
 		(fields_autoplaced yes)
-		(property "Reference" "#PWR0294"
+		(property "Reference" "#PWR0290"
 			(at 217.17 128.27 0)
 			(effects
@@
 			(project "arb"
 				(path "/866ef9be-3b01-4288-a6e0-a2357aa17e50/dd20ed2c-105a-40ef-bdba-a4198899f68e"
-					(reference "#PWR0294")
+					(reference "#PWR0290")
 					(unit 1)
 				)
@@
 		(dnp no)
 		(fields_autoplaced yes)
-		(property "Reference" "#PWR0286"
+		(property "Reference" "#PWR0282"
 			(at 107.95 97.79 0)
 			(effects
@@
 			(project "arb"
 				(path "/866ef9be-3b01-4288-a6e0-a2357aa17e50/dd20ed2c-105a-40ef-bdba-a4198899f68e"
-					(reference "#PWR0286")
-					(unit 1)
-				)
+					(reference "#PWR0282")
+					(unit 1)
+				)

Commit message: FEAT: Routed Analog and all Misc Signals. Routing is complete.
Parts:
- renumbered R85 to R87, R86 to R88, R87 to R89, R88 to R90, R89 to R91, R90 to R92
Changed lines of the file:
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@@
 		(dnp no)
 		(fields_autoplaced yes)
-		(property "Reference" "R90"
+		(property "Reference" "R92"
 			(at 186.69 110.4899 0)
 			(effects
@@
 			(project "arb"
 				(path "/866ef9be-3b01-4288-a6e0-a2357aa17e50/dd20ed2c-105a-40ef-bdba-a4198899f68e"
-					(reference "R90")
+					(reference "R92")
 					(unit 1)
 				)
@@
 		(dnp no)
 		(fields_autoplaced yes)
-		(property "Reference" "R87"
+		(property "Reference" "R89"
 			(at 92.71 107.9499 0)
 			(effects
@@
 			(project "arb"
 				(path "/866ef9be-3b01-4288-a6e0-a2357aa17e50/dd20ed2c-105a-40ef-bdba-a4198899f68e"
-					(reference "R87")
+					(reference "R89")
 					(unit 1)
 				)
@@
 		(on_board yes)
 		(dnp no)
-		(property "Reference" "R86"
+		(property "Reference" "R88"
 			(at 78.74 108.204 90)
 			(effects
@@
 			(project "arb"
 				(path "/866ef9be-3b01-4288-a6e0-a2357aa17e50/dd20ed2c-105a-40ef-bdba-a4198899f68e"
-					(reference "R86")
+					(reference "R88")
 					(unit 1)
 				)
@@
 		(dnp no)
 		(fields_autoplaced yes)
-		(property "Reference" "R88"
+		(property "Reference" "R90"
 			(at 106.68 69.85 90)
 			(effects
@@
 			(project "arb"
 				(path "/866ef9be-3b01-4288-a6e0-a2357aa17e50/dd20ed2c-105a-40ef-bdba-a4198899f68e"
-					(reference "R88")
+					(reference "R90")
 					(unit 1)
 				)
@@
 		(on_board yes)
 		(dnp no)
-		(property "Reference" "R85"
+		(property "Reference" "R87"
 			(at 78.74 93.98 90)
 			(effects
@@
 			(project "arb"
 				(path "/866ef9be-3b01-4288-a6e0-a2357aa17e50/dd20ed2c-105a-40ef-bdba-a4198899f68e"
-					(reference "R85")
+					(reference "R87")
 					(unit 1)
 				)
@@
 		(dnp no)
 		(fields_autoplaced yes)
-		(property "Reference" "R89"
+		(property "Reference" "R91"
 			(at 127 96.52 90)
 			(effects
@@
 			(project "arb"
 				(path "/866ef9be-3b01-4288-a6e0-a2357aa17e50/dd20ed2c-105a-40ef-bdba-a4198899f68e"
-					(reference "R89")
-					(unit 1)
-				)
+					(reference "R91")
+					(unit 1)
+				)
