File: 2_HARDWARE/03_PCB/connectors.kicad_sch (KiCad schematic)
At the start: 19 parts, among them J1 TYPE-C-31-M-12, J2 SMA, J3 SMA, J4 BNC, J5 PH-00244

Commit message: FEAT: Removed Via in Pad from Design + added sitching vias.
Parts:
- H1: footprint MountingHole:MountingHole_3.2mm_M3_Pad_TopBottom -> MountingHole:MountingHole_3.2mm_M3_Pad_Via
Changed lines of the file:
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@@
 			)
 		)
-		(property "Footprint" "MountingHole:MountingHole_3.2mm_M3_Pad_TopBottom"
+		(property "Footprint" "MountingHole:MountingHole_3.2mm_M3_Pad_Via"
 			(at 232.41 17.78 0)
 			(effects
